Commit message: CHANGE: name of joints in controller yaml

File: fingrip_moveit_config/srdf/fingrip_arm.xacro (robot description, xacro)
@@ -14,11 +14,11 @@
     <!-- Can configurate pos -->
     <group_state group="arm" name="ready">
-      <joint name="${prefix}joint1" value="0"/>
-      <joint name="${prefix}joint2" value="${-pi/4}"/>
-      <joint name="${prefix}joint3" value="0"/>
-      <joint name="${prefix}joint4" value="${-135*pi/180}"/>
-      <joint name="${prefix}joint5" value="0"/>
-      <joint name="${prefix}joint6" value="${pi/2}"/>
-      <joint name="${prefix}joint7" value="${pi/4}"/>
+      <joint name="${prefix}joint1" value="${108*pi/180}"/>
+      <joint name="${prefix}joint2" value="${-35*pi/180}"/>
+      <joint name="${prefix}joint3" value="${154*pi/180}"/>
+      <joint name="${prefix}joint4" value="${88*pi/180}"/>
+      <joint name="${prefix}joint5" value="${-72*pi/180}"/>
+      <joint name="${prefix}joint6" value="${-100*pi/180}"/>
+      <joint name="${prefix}joint7" value="${-125*pi/180}"/>
     </group_state>
     <group_state group="arm" name="extended">
@@ -31,5 +31,5 @@
       <joint name="${prefix}joint7" value="0"/>
     </group_state>
-    <group_state group="arm" name="transport">
+    <!-- <group_state group="arm" name="transport">
       <joint name="${prefix}joint1" value="0"/>
       <joint name="${prefix}joint2" value="${-32.08*pi/180}"/>
@@ -39,5 +39,5 @@
       <joint name="${prefix}joint6" value="0"/>
       <joint name="${prefix}joint7" value="${pi/4}"/>
-    </group_state>
+    </group_state> -->
     <disable_collisions link1="${prefix}link0" link2="${prefix}link1" reason="Adjacent"/>
     <disable_collisions link1="${prefix}link0" link2="${prefix}link2" reason="Never"/>
