Commit message: UPD: passage de panda à fingrip au niveau des arguments...

File: fingrip_description/urdf/fingrip.urdf (robot description, URDF)
Before this commit: robot panda, 14 links, 13 joints
Links:
- removed link panda_hand
- removed link panda_hand_tcp
- removed link panda_leftfinger
- removed link panda_link0
- removed link panda_link1
- removed link panda_link2
- removed link panda_link3
- removed link panda_link4
- removed link panda_link5
- removed link panda_link6
- removed link panda_link7
- removed link panda_link8
- removed link panda_rightfinger
- added link fingrip_hand, mass 0.14060765127978503; collision mesh filename=package://fingrip_description/meshes/collision/hand.stl; visual mesh filename=package://fingrip_description/meshes/visual/hand.dae
- added link fingrip_hand_tcp
- added link fingrip_leftfinger, mass 0.2238453537819424; collision mesh filename=package://fingrip_description/meshes/collision/finger.stl; visual mesh filename=package://fingrip_description/meshes/visual/finger.dae
- added link fingrip_link0, mass 2.814271300104062; collision mesh filename=package://fingrip_description/meshes/collision/link0.stl; visual mesh filename=package://fingrip_description/meshes/visual/link0.dae
- added link fingrip_link1, mass 2.6433170427227215; collision mesh filename=package://fingrip_description/meshes/collision/link1.stl; visual mesh filename=package://fingrip_description/meshes/visual/link1.dae
- added link fingrip_link2, mass 2.6652755331661186; collision mesh filename=package://fingrip_description/meshes/collision/link2.stl; visual mesh filename=package://fingrip_description/meshes/visual/link2.dae
- added link fingrip_link3, mass 2.3293714829045733; collision mesh filename=package://fingrip_description/meshes/collision/link3.stl; visual mesh filename=package://fingrip_description/meshes/visual/link3.dae
- added link fingrip_link4, mass 2.3104763646281508; collision mesh filename=package://fingrip_description/meshes/collision/link4.stl; visual mesh filename=package://fingrip_description/meshes/visual/link4.dae
- added link fingrip_link5, mass 2.6226426154892004; collision mesh filename=package://fingrip_description/meshes/collision/link5.stl; visual mesh filename=package://fingrip_description/meshes/visual/link5.dae
- added link fingrip_link6, mass 1.5025804886626795; collision mesh filename=package://fingrip_description/meshes/collision/link6.stl; visual mesh filename=package://fingrip_description/meshes/visual/link6.dae
- added link fingrip_link7, mass 0.5237668134788256; collision mesh filename=package://fingrip_description/meshes/collision/link7.stl; visual mesh filename=package://fingrip_description/meshes/visual/link7.dae
- added link fingrip_link8
- added link fingrip_rightfinger, mass 0.2238453537819424; collision mesh filename=package://fingrip_description/meshes/collision/finger.stl; visual mesh filename=package://fingrip_description/meshes/visual/finger.dae
Joints:
- removed joint panda_finger_joint1
- removed joint panda_finger_joint2
- removed joint panda_hand_tcp_virtual_joint
- removed joint panda_joint1
- removed joint panda_joint2
- removed joint panda_joint3
- removed joint panda_joint4
- removed joint panda_joint5
- removed joint panda_joint6
- removed joint panda_joint7
- removed joint panda_joint_base
- removed joint panda_joint_wrist
- removed joint panda_link8_virtual_joint
- added joint fingrip_finger_joint1: type prismatic, parent fingrip_hand, child fingrip_leftfinger, origin xyz=0 0 0.0584 rpy=0 0 0, axis 0 1 0, limit lower=0 upper=0.04 effort=20 velocity=0.2
- added joint fingrip_finger_joint2: type prismatic, parent fingrip_hand, child fingrip_rightfinger, origin xyz=0 0 0.0584 rpy=0 0 0, axis 0 -1 0, limit lower=0 upper=0.04 effort=20 velocity=0.2
- added joint fingrip_hand_tcp_virtual_joint: type fixed, parent fingrip_hand, child fingrip_hand_tcp, origin xyz=0 0 0.1034 rpy=0 0 0
- added joint fingrip_joint1: type revolute, parent fingrip_link0, child fingrip_link1, origin xyz=0 0 0.333 rpy=0 0 0, axis 0 0 1, limit lower=-2.897246558310587 upper=2.897246558310587 effort=87 velocity=2.6179938779914944
- added joint fingrip_joint2: type revolute, parent fingrip_link1, child fingrip_link2, origin xyz=0 0 0 rpy=-1.5707963267948966 0 0, axis 0 0 1, limit lower=-1.7627825445142729 upper=1.7627825445142729 effort=87 velocity=2.6179938779914944
- added joint fingrip_joint3: type revolute, parent fingrip_link2, child fingrip_link3, origin xyz=0 -0.316 0 rpy=1.5707963267948966 0 0, axis 0 0 1, limit lower=-2.897246558310587 upper=2.897246558310587 effort=87 velocity=2.6179938779914944
- added joint fingrip_joint4: type revolute, parent fingrip_link3, child fingrip_link4, origin xyz=0.0825 0 0 rpy=1.5707963267948966 0 0, axis 0 0 1, limit lower=-3.07177948351002 upper=-0.06981317007977318 effort=87 velocity=2.6179938779914944
- added joint fingrip_joint5: type revolute, parent fingrip_link4, child fingrip_link5, origin xyz=-0.0825 0.384 0 rpy=-1.5707963267948966 0 0, axis 0 0 1, limit lower=-2.897246558310587 upper=2.897246558310587 effort=12 velocity=3.141592653589793
- added joint fingrip_joint6: type revolute, parent fingrip_link5, child fingrip_link6, origin xyz=0 0 0 rpy=1.5707963267948966 0 0, axis 0 0 1, limit lower=-0.017453292519943295 upper=3.752457891787808 effort=12 velocity=3.141592653589793
- added joint fingrip_joint7: type revolute, parent fingrip_link6, child fingrip_link7, origin xyz=0.088 0 0 rpy=1.5707963267948966 0 0, axis 0 0 1, limit lower=-2.897246558310587 upper=2.897246558310587 effort=12 velocity=3.141592653589793
- added joint fingrip_joint_base: type fixed, parent world, child fingrip_link0, origin xyz=0 0 0 rpy=0 0 0
- added joint fingrip_joint_wrist: type fixed, parent fingrip_link8, child fingrip_hand, origin xyz=0 0 0 rpy=0 0 0
- added joint fingrip_link8_virtual_joint: type fixed, parent fingrip_link7, child fingrip_link8, origin xyz=0 0 0.107 rpy=0 0 -0.7853981633974483

File: fingrip_description/urdf/fingrip.urdf.xacro (robot description, xacro)
@@ -1,17 +1,17 @@
 <?xml version="1.0"?>
-<!-- URDF for Franka Emika Panda -->
+<!-- URDF for Franka Emika fingrip -->
 <robot xmlns:xacro="http://wiki.ros.org/xacro" name="$(arg name)">
   <!--                   -->
   <!-- Imported elements -->
   <!--                   -->
-  <xacro:include filename="$(find panda_description)/urdf/panda_arm.xacro"/>
-  <xacro:include filename="$(find panda_description)/urdf/panda_gripper.xacro"/>
-  <xacro:include filename="$(find panda_description)/urdf/panda_utils.xacro"/>
-  <xacro:include filename="$(find panda_description)/urdf/panda.gazebo"/>
+  <xacro:include filename="$(find fingrip_description)/urdf/fingrip_arm.xacro"/>
+  <xacro:include filename="$(find fingrip_description)/urdf/fingrip_gripper.xacro"/>
+  <xacro:include filename="$(find fingrip_description)/urdf/fingrip_utils.xacro"/>
+  <xacro:include filename="$(find fingrip_description)/urdf/fingrip.gazebo"/>
   <!--            -->
   <!-- Parameters -->
   <!--            -->
   <!-- Name of the robot (mandatory) -->
-  <xacro:arg name="name" default="panda"/>
+  <xacro:arg name="name" default="fingrip"/>
   <!-- Prefix for all entities -->
   <xacro:arg name="prefix" default="$(arg name)_"/>
@@ -37,5 +37,5 @@
   <xacro:arg name="ros2_control_command_interface" default="effort"/>
   <!-- The filepath to parameters of ROS 2 controllers -->
-  <xacro:arg name="ros2_controller_parameters" default="$(find panda_moveit_config)/config/controllers_$(arg ros2_control_command_interface).yaml"/>
+  <xacro:arg name="ros2_controller_parameters" default="$(find fingrip_moveit_config)/config/controllers_$(arg ros2_control_command_interface).yaml"/>
   <!-- Flag to preserve fixed joints and prevent lumping when generating SDF for Gazebo -->
   <xacro:arg name="gazebo_preserve_fixed_joint" default="false"/>
@@ -57,10 +57,10 @@
   <!--       -->
   <!-- Dummy world link that the robot is fixed to -->
-  <xacro:panda_dummy_link
+  <xacro:fingrip_dummy_link
     link_name="${world_name}"
     gazebo_preserve_fixed_joint="$(arg gazebo_preserve_fixed_joint)"
   />
   <!-- Arm -->
-  <xacro:panda_arm
+  <xacro:fingrip_arm
     base_parent="world"
     prefix="${prefix_arm}"
@@ -79,5 +79,5 @@
   <!-- Gripper -->
   <xacro:if value="$(arg gripper)">
-    <xacro:panda_gripper
+    <xacro:fingrip_gripper
       wrist_flange="${prefix_arm}${wrist_flange_name}"
       prefix="${prefix_gripper}"

File: fingrip_description/urdf/fingrip_arm.xacro (robot description, xacro)
@@ -1,10 +1,10 @@
 <?xml version="1.0"?>
-<!-- Xacro for Franka Emika Panda arm -->
+<!-- Xacro for Franka Emika fingrip arm -->
 <robot xmlns:xacro="http://www.ros.org/wiki/xacro">
   <!--                   -->
   <!-- Imported elements -->
   <!--                   -->
-  <xacro:include filename="$(find panda_description)/urdf/panda_utils.xacro"/>
-  <xacro:include filename="$(find panda_description)/urdf/panda.ros2_control"/>
+  <xacro:include filename="$(find fingrip_description)/urdf/fingrip_utils.xacro"/>
+  <xacro:include filename="$(find fingrip_description)/urdf/fingrip.ros2_control"/>
   <!--            -->
   <!-- Properties -->
@@ -113,7 +113,7 @@
   <xacro:property name="default_origin_xyz" value="0 0 0"/>
   <xacro:property name="default_origin_rpy" value="0 0 0"/>
-  <xacro:macro name="panda_arm" params="
+  <xacro:macro name="fingrip_arm" params="
     base_parent
-    prefix:=panda_
+    prefix:=fingrip_
     origin_xyz:=${default_origin_xyz}
     origin_rpy:=${default_origin_rpy}
@@ -129,5 +129,5 @@
   ">
     <!-- Base -->
-    <xacro:panda_joint
+    <xacro:fingrip_joint
     parent="${base_parent}"
     child="${prefix}${link0_name}"
@@ -138,5 +138,5 @@
     gazebo_preserve_fixed_joint="${gazebo_preserve_fixed_joint}"
     />
-    <xacro:panda_link
+    <xacro:fingrip_link
     link_name="${prefix}${link0_name}"
     mesh="${link0_mesh}"
@@ -145,5 +145,5 @@
     />
     <!-- 1 -->
-    <xacro:panda_joint
+    <xacro:fingrip_joint
     parent="${prefix}${link0_name}"
     child="${prefix}${link1_name}"
@@ -165,5 +165,5 @@
     gazebo_preserve_fixed_joint="${gazebo_preserve_fixed_joint}"
     />
-    <xacro:panda_link
+    <xacro:fingrip_link
     link_name="${prefix}${link1_name}"
     mesh="${link1_mesh}"
@@ -172,5 +172,5 @@
     />
     <!-- 2 -->
-    <xacro:panda_joint
+    <xacro:fingrip_joint
     parent="${prefix}${link1_name}"
     child="${prefix}${link2_name}"
@@ -192,5 +192,5 @@
     gazebo_preserve_fixed_joint="${gazebo_preserve_fixed_joint}"
     />
-    <xacro:panda_link
+    <xacro:fingrip_link
     link_name="${prefix}${link2_name}"
     mesh="${link2_mesh}"
@@ -199,5 +199,5 @@
     />
     <!-- 3 -->
-    <xacro:panda_joint
+    <xacro:fingrip_joint
     parent="${prefix}${link2_name}"
     child="${prefix}${link3_name}"
@@ -219,5 +219,5 @@
     gazebo_preserve_fixed_joint="${gazebo_preserve_fixed_joint}"
     />
-    <xacro:panda_link
+    <xacro:fingrip_link
     link_name="${prefix}${link3_name}"
     mesh="${link3_mesh}"
@@ -226,5 +226,5 @@
     />
     <!-- 4 -->
-    <xacro:panda_joint
+    <xacro:fingrip_joint
     parent="${prefix}${link3_name}"
     child="${prefix}${link4_name}"
@@ -246,5 +246,5 @@
     gazebo_preserve_fixed_joint="${gazebo_preserve_fixed_joint}"
     />
-    <xacro:panda_link
+    <xacro:fingrip_link
     link_name="${prefix}${link4_name}"
     mesh="${link4_mesh}"
@@ -253,5 +253,5 @@
     />
     <!-- 5 -->
-    <xacro:panda_joint
+    <xacro:fingrip_joint
     parent="${prefix}${link4_name}"
     child="${prefix}${link5_name}"
@@ -273,5 +273,5 @@
     gazebo_preserve_fixed_joint="${gazebo_preserve_fixed_joint}"
     />
-    <xacro:panda_link
+    <xacro:fingrip_link
     link_name="${prefix}${link5_name}"
     mesh="${link5_mesh}"
@@ -280,5 +280,5 @@
     />
     <!-- 6 -->
-    <xacro:panda_joint
+    <xacro:fingrip_joint
     parent="${prefix}${link5_name}"
     child="${prefix}${link6_name}"
@@ -300,5 +300,5 @@
     gazebo_preserve_fixed_joint="${gazebo_preserve_fixed_joint}"
     />
-    <xacro:panda_link
+    <xacro:fingrip_link
     link_name="${prefix}${link6_name}"
     mesh="${link6_mesh}"
@@ -307,5 +307,5 @@
     />
     <!-- 7 -->
-    <xacro:panda_joint
+    <xacro:fingrip_joint
     parent="${prefix}${link6_name}"
     child="${prefix}${link7_name}"
@@ -327,5 +327,5 @@
     gazebo_preserve_fixed_joint="${gazebo_preserve_fixed_joint}"
     />
-    <xacro:panda_link
+    <xacro:fingrip_link
     link_name="${prefix}${link7_name}"
     mesh="${link7_mesh}"
@@ -334,5 +334,5 @@
     />
     <!-- Wrist flange -->
-    <xacro:panda_virtual_link
+    <xacro:fingrip_virtual_link
     parent="${prefix}${link7_name}"
     link_name="${prefix}${wrist_flange_name}"
@@ -343,5 +343,5 @@
     <!-- ROS 2 control -->
     <xacro:if value="${ros2_control}">
-      <xacro:ros2_control_panda_arm prefix="${prefix}" plugin="${ros2_control_plugin}" command_interface="${ros2_control_command_interface}"/>
+      <xacro:ros2_control_fingrip_arm prefix="${prefix}" plugin="${ros2_control_plugin}" command_interface="${ros2_control_command_interface}"/>
     </xacro:if>
   </xacro:macro>

File: fingrip_description/urdf/fingrip_gripper.xacro (robot description, xacro)
@@ -1,10 +1,10 @@
 <?xml version="1.0"?>
-<!-- Xacro for Franka Emika Panda gripper -->
+<!-- Xacro for Franka Emika fingrip gripper -->
 <robot xmlns:xacro="http://www.ros.org/wiki/xacro">
   <!--                   -->
   <!-- Imported elements -->
   <!--                   -->
-  <xacro:include filename="$(find panda_description)/urdf/panda_utils.xacro"/>
-  <xacro:include filename="$(find panda_description)/urdf/panda.ros2_control"/>
+  <xacro:include filename="$(find fingrip_description)/urdf/fingrip_utils.xacro"/>
+  <xacro:include filename="$(find fingrip_description)/urdf/fingrip.ros2_control"/>
   <!--            -->
   <!-- Properties -->
@@ -50,7 +50,7 @@
   <xacro:property name="default_origin_xyz" value="0 0 0"/>
   <xacro:property name="default_origin_rpy" value="0 0 0"/>
-  <xacro:macro name="panda_gripper" params="
+  <xacro:macro name="fingrip_gripper" params="
     wrist_flange
-    prefix:=panda_
+    prefix:=fingrip_
     origin_xyz:=${default_origin_xyz}
     origin_rpy:=${default_origin_rpy}
@@ -62,5 +62,5 @@
   ">
     <!-- Wrist -->
-    <xacro:panda_joint
+    <xacro:fingrip_joint
     parent="${wrist_flange}"
     child="${prefix}${hand_name}"
@@ -71,5 +71,5 @@
     gazebo_preserve_fixed_joint="${gazebo_preserve_fixed_joint}"
     />
-    <xacro:panda_link
+    <xacro:fingrip_link
     link_name="${prefix}${hand_name}"
     mesh="${hand_mesh}"
@@ -78,5 +78,5 @@
     />
     <!-- Finger 1 -->
-    <xacro:panda_joint
+    <xacro:fingrip_joint
     parent="${prefix}${hand_name}"
     child="${prefix}${link_finger1_name}"
@@ -94,5 +94,5 @@
     gazebo_preserve_fixed_joint="${gazebo_preserve_fixed_joint}"
     />
-    <xacro:panda_link
+    <xacro:fingrip_link
     link_name="${prefix}${link_finger1_name}"
     mesh="${finger_mesh}"
@@ -102,5 +102,5 @@
     />
     <!-- Finger 2 -->
-    <xacro:panda_joint
+    <xacro:fingrip_joint
     parent="${prefix}${hand_name}"
     child="${prefix}${link_finger2_name}"
@@ -118,5 +118,5 @@
     gazebo_preserve_fixed_joint="${gazebo_preserve_fixed_joint}"
     />
-    <xacro:panda_link
+    <xacro:fingrip_link
     link_name="${prefix}${link_finger2_name}"
     mesh="${finger_mesh}"
@@ -126,5 +126,5 @@
     />
     <!-- End effector -->
-    <xacro:panda_virtual_link
+    <xacro:fingrip_virtual_link
     parent="${prefix}${hand_name}"
     link_name="${prefix}${ee_name}"
@@ -135,5 +135,5 @@
     <!-- ROS 2 control -->
     <xacro:if value="${ros2_control}">
-      <xacro:ros2_control_panda_gripper prefix="${prefix}" plugin="${ros2_control_plugin}" command_interface="${ros2_control_command_interface}"/>
+      <xacro:ros2_control_fingrip_gripper prefix="${prefix}" plugin="${ros2_control_plugin}" command_interface="${ros2_control_command_interface}"/>
     </xacro:if>
   </xacro:macro>

File: fingrip_description/urdf/fingrip_inertial.xacro (robot description, xacro)
@@ -1,4 +1,4 @@
 <?xml version="1.0"?>
-<!-- Macro for inertial properties of Franka Emika Panda -->
+<!-- Macro for inertial properties of Franka Emika fingrip -->
 <robot xmlns:xacro="http://www.ros.org/wiki/xacro">
   <!--            -->
@@ -19,5 +19,5 @@
   <!--       -->
   <xacro:property name="mesh_offset_rpy" value="0 0 0"/>
-  <xacro:macro name="panda_inertial" params="
+  <xacro:macro name="fingrip_inertial" params="
     mesh
     mesh_offset_rpy:=${mesh_offset_rpy}

File: fingrip_description/urdf/fingrip_utils.xacro (robot description, xacro)
@@ -5,10 +5,10 @@
   <!-- Imported elements -->
   <!--                   -->
-  <xacro:include filename="$(find panda_description)/urdf/panda_inertial.xacro"/>
+  <xacro:include filename="$(find fingrip_description)/urdf/fingrip_inertial.xacro"/>
   <!--       -->
   <!-- Macro -->
   <!--       -->
   <xacro:property name="mesh_offset_rpy" value="0 0 0"/>
-  <xacro:macro name="panda_link" params="
+  <xacro:macro name="fingrip_link" params="
     link_name
     mesh
@@ -22,5 +22,5 @@
         <origin xyz="0 0 0" rpy="${mesh_offset_rpy}"/>
         <geometry>
-          <mesh filename="package://panda_description/meshes/visual/${mesh}.dae"/>
+          <mesh filename="package://fingrip_description/meshes/visual/${mesh}.dae"/>
         </geometry>
       </visual>
@@ -29,9 +29,9 @@
           <origin xyz="0 0 0" rpy="${mesh_offset_rpy}"/>
           <geometry>
-            <mesh filename="package://panda_description/meshes/collision/${mesh}.stl"/>
+            <mesh filename="package://fingrip_description/meshes/collision/${mesh}.stl"/>
           </geometry>
         </collision>
       </xacro:if>
-      <xacro:panda_inertial mesh="${mesh}" mesh_offset_rpy="${mesh_offset_rpy}"/>
+      <xacro:fingrip_inertial mesh="${mesh}" mesh_offset_rpy="${mesh_offset_rpy}"/>
     </link>
     <gazebo reference="${link_name}">
@@ -46,5 +46,5 @@
   <!-- Macro -->
   <!--       -->
-  <xacro:macro name="panda_joint" params="
+  <xacro:macro name="fingrip_joint" params="
     parent
     child
@@ -138,5 +138,5 @@
   <!-- Macro -->
   <!--       -->
-  <xacro:macro name="panda_virtual_link" params="
+  <xacro:macro name="fingrip_virtual_link" params="
     parent
     link_name
@@ -145,5 +145,5 @@
     gazebo_preserve_fixed_joint:=false
   ">
-    <xacro:panda_dummy_link
+    <xacro:fingrip_dummy_link
       link_name="${link_name}"
       gazebo_preserve_fixed_joint="${gazebo_preserve_fixed_joint}"
@@ -158,5 +158,5 @@
   <!-- Macro -->
   <!--       -->
-  <xacro:macro name="panda_dummy_link" params="
+  <xacro:macro name="fingrip_dummy_link" params="
     link_name
     gazebo_preserve_fixed_joint:=false

File: fingrip_moveit_config/srdf/fingrip.srdf.xacro (robot description, xacro)
@@ -1,4 +1,4 @@
 <?xml version="1.0"?>
-<!-- SRDF for Franka Emika Panda -->
+<!-- SRDF for Franka Emika fingrip -->
 <robot xmlns:xacro="http://wiki.ros.org/xacro" name="$(arg name)">
   <!--                   -->

File: fingrip_moveit_config/srdf/fingrip_arm.xacro (robot description, xacro)
@@ -1,4 +1,4 @@
 <?xml version="1.0"?>
-<!-- Macro for SRDF of Franka Emika Panda arm -->
+<!-- Macro for SRDF of Franka Emika fingrip arm -->
 <robot xmlns:xacro="http://wiki.ros.org/xacro">
   <!--       -->

File: fingrip_moveit_config/srdf/fingrip_gripper.xacro (robot description, xacro)
@@ -1,4 +1,4 @@
 <?xml version="1.0"?>
-<!-- Macro for SRDF of Franka Emika Panda gripper -->
+<!-- Macro for SRDF of Franka Emika fingrip gripper -->
 <robot xmlns:xacro="http://www.ros.org/wiki/xacro">
   <!--       -->
