Commit message: ADD: proximal limbs for fingers + Add srdf file for moveit commander

File: fingrip_description/urdf/fingrip.urdf (robot description, URDF)
Before this commit: robot fingrip, 16 links, 15 joints
Links:
- added link fingrip_finger1_proximal_link, mass 0.2238453537819424; collision mesh filename=package://fingrip_description/meshes/collision/gripper/prox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; visual mesh filename=package://fingrip_description/meshes/visual/gripper/proxima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
- added link fingrip_finger2_proximal_link, mass 0.2238453537819424; collision mesh filename=package://fingrip_description/meshes/collision/gripper/prox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; visual mesh filename=package://fingrip_description/meshes/visual/gripper/proxima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
- added link fingrip_finger3_proximal_link, mass 0.2238453537819424; collision mesh filename=package://fingrip_description/meshes/collision/gripper/prox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; visual mesh filename=package://fingrip_description/meshes/visual/gripper/proxima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
Joints:
- added joint fingrip_finger1_proximal_joint: type revolute, parent fingrip_finger1_base_link, child fingrip_finger1_proximal_link, origin xyz=0 -0.03255 0 rpy=0 0 0, axis 0 0 1, limit lower=-1.3 upper=0.31416 effort=20 velocity=0.2
- added joint fingrip_finger2_proximal_joint: type revolute, parent fingrip_finger2_base_link, child fingrip_finger2_proximal_link, origin xyz=0 -0.03255 0 rpy=0 0 0, axis 0 0 1, limit lower=-1.3 upper=0.31416 effort=20 velocity=0.2
- added joint fingrip_finger3_proximal_joint: type revolute, parent fingrip_finger3_base_link, child fingrip_finger3_proximal_link, origin xyz=0 -0.03255 0 rpy=0 0 0, axis 0 0 1, limit lower=-1.3 upper=0.31416 effort=20 velocity=0.2

File: fingrip_description/urdf/fingrip_finger.xacro (robot description, xacro)
@@ -28,7 +28,7 @@
   <xacro:property name="joint_proximal_lower_limit" value="-1.3"/>
   <xacro:property name="joint_proximal_upper_limit" value="0.31416"/>
-  <xacro:property name="joint_proximal_origin_xyz" value="0 0 0.0584"/>
+  <xacro:property name="joint_proximal_origin_xyz" value="0 -0.03255 0"/>
   <xacro:property name="joint_proximal_origin_rpy" value="0 0 0"/>
-  <xacro:property name="joint_proximal_axis_xyz" value="0 1 0"/>
+  <xacro:property name="joint_proximal_axis_xyz" value="0 0 1"/>
   <!-- Intermediaire -->
   <xacro:property name="joint_intermediaire_lower_limit" value="-0.5"/>
@@ -36,5 +36,5 @@
   <xacro:property name="joint_intermediaire_origin_xyz" value="0 0 0.0584"/>
   <xacro:property name="joint_intermediaire_origin_rpy" value="0 0 0"/>
-  <xacro:property name="joint_intermediaire_axis_xyz" value="0 1 0"/>
+  <xacro:property name="joint_intermediaire_axis_xyz" value="0 0 1"/>
   <!-- Distal -->
   <xacro:property name="joint_distal_lower_limit" value="-0.5"/>
@@ -42,5 +42,5 @@
   <xacro:property name="joint_distal_origin_xyz" value="0 0 0.0584"/>
   <xacro:property name="joint_distal_origin_rpy" value="0 0 0"/>
-  <xacro:property name="joint_distal_axis_xyz" value="0 1 0"/>
+  <xacro:property name="joint_distal_axis_xyz" value="0 0 1"/>
   <!--       -->
   <!-- Macro -->
@@ -88,5 +88,4 @@
         />
         <!-- PROXIMAL limb -->
-        <!--
         <xacro:fingrip_joint
         parent="${prefix}${finger_name}${base_prefix}${link_prefix}"
@@ -94,7 +93,7 @@
         joint_name="${prefix}${finger_name}${proximal_prefix}${joint_prefix}"
         joint_type="${joint_other_type}"
-        joint_origin_xyz="${joint_origin_xyz}"
-        joint_origin_rpy="${joint_origin_rpy}"
-        joint_axis_xyz="${joint_axis_xyz}"
+        joint_origin_xyz="${joint_proximal_origin_xyz}"
+        joint_origin_rpy="${joint_proximal_origin_rpy}"
+        joint_axis_xyz="${joint_proximal_axis_xyz}"
         joint_lower_limit="${joint_proximal_lower_limit}"
         joint_upper_limit="${joint_proximal_upper_limit}"
@@ -112,5 +111,4 @@
         mesh_offset_rpy="${mesh_offset_rpy}"
         />
-        -->
         <!-- INTERMEDIAIRE limb -->
         <!--

File: fingrip_description/urdf/fingrip_gripper.xacro (robot description, xacro)
@@ -99,5 +99,5 @@
         joint_lower_limit="${-joint_base_upper_limit}"
         joint_upper_limit="${-joint_base_lower_limit}"
-        gazebo_preserve_fixed_joint="${gazebo_preserve_fixed_joint}"
+        gazebo_preserve_fixed_joint="true"
         />
         <!-- FINGER 2 -->
@@ -112,5 +112,5 @@
         joint_origin_rpy="${joint_finger2_base_origin_rpy}"
         joint_axis_xyz="${joint_finger2_base_axis_xyz}"
-        gazebo_preserve_fixed_joint="${gazebo_preserve_fixed_joint}"
+        gazebo_preserve_fixed_joint="true"
         />
         <!-- FINGER 3 -->
@@ -125,5 +125,5 @@
         joint_origin_rpy="${joint_finger3_base_origin_rpy}"
         joint_axis_xyz="${joint_finger3_base_axis_xyz}"
-        gazebo_preserve_fixed_joint="${gazebo_preserve_fixed_joint}"
+        gazebo_preserve_fixed_joint="true"
         />
         <!-- FINGER 4 -->
@@ -139,5 +139,5 @@
             joint_origin_rpy="${joint_finger4_base_origin_rpy}"
             joint_axis_xyz="${joint_finger4_base_axis_xyz}"
-            gazebo_preserve_fixed_joint="${gazebo_preserve_fixed_joint}"
+            gazebo_preserve_fixed_joint="true"
             />
         </xacro:unless>
@@ -157,11 +157,14 @@
         plugin="${ros2_control_plugin}"
         command_interface="${ros2_control_command_interface}"
-        finger_name="${finger1_name}"/>
+        finger_name="${finger1_name}"
+        abduction="true"
+        />
         <xacro:ros2_control_fingrip_gripper
         prefix="${prefix}"
         plugin="${ros2_control_plugin}"
         command_interface="${ros2_control_command_interface}"
-        finger_name="${finger2_name}"/>
-        <!--
+        finger_name="${finger2_name}"
+        abduction="true"
+        />
         <xacro:ros2_control_fingrip_gripper
         prefix="${prefix}"
@@ -169,5 +172,4 @@
         command_interface="${ros2_control_command_interface}"
         finger_name="${finger3_name}"/>
-        -->
         <xacro:unless value="${nbFingers == 3}">
           <xacro:ros2_control_fingrip_gripper

File: fingrip_description/urdf/fingrip_inertial.xacro (robot description, xacro)
@@ -118,5 +118,5 @@
     <xacro:if value="${mesh == case_mesh_path+'3d'}">
       <inertial>
-        <origin xyz="-6.7624e-06 0.00152435 0.0275912" rpy="${mesh_offset_rpy}"/>
+        <origin xyz="0 0 0.0" rpy="${mesh_offset_rpy}"/>
         <mass value="0.14060765127978503"/>
         <inertia ixx="0.0005365450414352072" iyy="7.70511954783727e-05" izz="0.0004938176882694914" ixy="1.7911952957732454e-08" ixz="-2.320071910601251e-08" iyz="4.681149945315967e-08"/>
@@ -125,5 +125,5 @@
     <xacro:if value="${mesh == case_mesh_path+'4d'}">
       <inertial>
-        <origin xyz="-6.7624e-06 0.00152435 0.0275912" rpy="${mesh_offset_rpy}"/>
+        <origin xyz="0 0.0 0.0" rpy="${mesh_offset_rpy}"/>
         <mass value="0.14060765127978503"/>
         <inertia ixx="0.0005365450414352072" iyy="7.70511954783727e-05" izz="0.0004938176882694914" ixy="1.7911952957732454e-08" ixz="-2.320071910601251e-08" iyz="4.681149945315967e-08"/>
@@ -133,7 +133,7 @@
     <xacro:if value="${mesh == base_mesh}">
       <inertial>
-        <origin xyz="-6.2561e-06 0.00227781 -0.0277116" rpy="${mesh_offset_rpy}"/>
+        <origin xyz="-0.0465 -0.04775 -0.0" rpy="${mesh_offset_rpy}"/>
         <mass value="0.2238453537819424"/>
-        <inertia ixx="6.74804167363695e-05" iyy="6.627189221641395e-05" izz="1.550396267804825e-05" ixy="-4.1027443646025676e-09" ixz="1.8693673970152995e-08" iyz="1.1967548474390802e-05"/>
+        <inertia ixx="0.0007" ixy="-0.0002" ixz="0.0" iyy="0.0006" iyz="0.0" izz="0.0011"/>
       </inertial>
     </xacro:if>
@@ -141,7 +141,7 @@
     <xacro:if value="${mesh == proximal_mesh_path+short_prefix+proximal_mesh_name}">
       <inertial>
-        <origin xyz="-6.2561e-06 0.00227781 -0.0277116" rpy="${mesh_offset_rpy}"/>
+        <origin xyz="0.03411 -0.01012 0.0" rpy="${mesh_offset_rpy}"/>
         <mass value="0.2238453537819424"/>
-        <inertia ixx="6.74804167363695e-05" iyy="6.627189221641395e-05" izz="1.550396267804825e-05" ixy="-4.1027443646025676e-09" ixz="1.8693673970152995e-08" iyz="1.1967548474390802e-05"/>
+        <inertia ixx="0.000092" ixy="-0.000061" ixz="0.0" iyy="0.00031" iyz="0.0" izz="0.00031"/>
       </inertial>
     </xacro:if>
@@ -149,7 +149,7 @@
     <xacro:if value="${mesh == intermediaire_mesh_path+short_prefix+intermediaire_mesh_name}">
       <inertial>
-        <origin xyz="-6.2561e-06 0.00227781 -0.0277116" rpy="${mesh_offset_rpy}"/>
+        <origin xyz="0.01791 -0.01023 0.0" rpy="${mesh_offset_rpy}"/>
         <mass value="0.2238453537819424"/>
-        <inertia ixx="6.74804167363695e-05" iyy="6.627189221641395e-05" izz="1.550396267804825e-05" ixy="-4.1027443646025676e-09" ixz="1.8693673970152995e-08" iyz="1.1967548474390802e-05"/>
+        <inertia ixx="0.000025" ixy="0.000013" ixz="0.0" iyy="0.000102" iyz="0.0" izz="0.000108"/>
       </inertial>
     </xacro:if>
@@ -157,7 +157,7 @@
     <xacro:if value="${mesh == distal_mesh_path+short_prefix+distal_mesh_name}">
       <inertial>
-        <origin xyz="-6.2561e-06 0.00227781 -0.0277116" rpy="${mesh_offset_rpy}"/>
+        <origin xyz="0.01217 -0.00732 0.0" rpy="${mesh_offset_rpy}"/>
         <mass value="0.2238453537819424"/>
-        <inertia ixx="6.74804167363695e-05" iyy="6.627189221641395e-05" izz="1.550396267804825e-05" ixy="-4.1027443646025676e-09" ixz="1.8693673970152995e-08" iyz="1.1967548474390802e-05"/>
+        <inertia ixx="0.000025" ixy="0.000013" ixz="0.0" iyy="0.000102" iyz="0.0" izz="0.000108"/>
       </inertial>
     </xacro:if>

File: fingrip_moveit_config/srdf/fingrip.srdf.xacro (robot description, xacro)
@@ -7,4 +7,5 @@
   <xacro:include filename="$(find fingrip_moveit_config)/srdf/fingrip_arm.xacro"/>
   <xacro:include filename="$(find fingrip_moveit_config)/srdf/fingrip_gripper.xacro"/>
+  <xacro:include filename="$(find fingrip_moveit_config)/srdf/fingrip_utils.xacro"/>
   <!--            -->
   <!-- Parameters -->
@@ -12,4 +13,7 @@
   <!-- Name of the robot (mandatory) -->
   <xacro:arg name="name" default="fingrip"/>
+  <xacro:arg name="nbFingers" default="3"/>
+  <xacro:arg name="nbArmjoints" default="7"/>
+  <xacro:arg name="nb_abduction_finger" default="2"/>
   <!-- Prefix for all entities -->
   <xacro:arg name="prefix" default="$(arg name)_"/>
@@ -25,9 +29,13 @@
   <xacro:fingrip_arm
     prefix="${prefix_arm}"
+    nbArmjoints="$(arg nbArmjoints)"
   />
   <xacro:fingrip_gripper
     prefix="${prefix_gripper}"
+    nbFingers="$(arg nbFingers)"
+    nb_abduction_finger="$(arg nb_abduction_finger)"
   />
   <end_effector group="gripper" name="gripper" parent_group="arm" parent_link="${prefix_arm}hand_tcp"/>
+  <!-- Palm And Hand -->
   <disable_collisions link1="${prefix_gripper}hand" link2="${prefix_arm}link3" reason="Never"/>
   <disable_collisions link1="${prefix_gripper}hand" link2="${prefix_arm}link4" reason="Never"/>
@@ -38,15 +46,9 @@
   <disable_collisions link1="${prefix_gripper}palm" link2="${prefix_arm}link6" reason="Never"/>
   <disable_collisions link1="${prefix_gripper}palm" link2="${prefix_arm}link7" reason="Never"/>
-  <disable_collisions link1="${prefix_gripper}finger1_base_link" link2="${prefix_arm}link3" reason="Never"/>
-  <disable_collisions link1="${prefix_gripper}finger1_base_link" link2="${prefix_arm}link4" reason="Never"/>
-  <disable_collisions link1="${prefix_gripper}finger1_base_link" link2="${prefix_arm}link6" reason="Never"/>
-  <disable_collisions link1="${prefix_gripper}finger1_base_link" link2="${prefix_arm}link7" reason="Never"/>
-  <disable_collisions link1="${prefix_gripper}finger2_base_link" link2="${prefix_arm}link3" reason="Never"/>
-  <disable_collisions link1="${prefix_gripper}finger2_base_link" link2="${prefix_arm}link4" reason="Never"/>
-  <disable_collisions link1="${prefix_gripper}finger2_base_link" link2="${prefix_arm}link6" reason="Never"/>
-  <disable_collisions link1="${prefix_gripper}finger2_base_link" link2="${prefix_arm}link7" reason="Never"/>
-  <disable_collisions link1="${prefix_gripper}finger3_base_link" link2="${prefix_arm}link3" reason="Never"/>
-  <disable_collisions link1="${prefix_gripper}finger3_base_link" link2="${prefix_arm}link4" reason="Never"/>
-  <disable_collisions link1="${prefix_gripper}finger3_base_link" link2="${prefix_arm}link6" reason="Never"/>
-  <disable_collisions link1="${prefix_gripper}finger3_base_link" link2="${prefix_arm}link7" reason="Never"/>
+  <!-- Fingers -->
+  <xacro:fingrip_gripper_arm_collision
+    prefix_gripper="${prefix_gripper}"
+    prefix_arm="${prefix_arm}"
+    nbFingers="$(arg nbFingers)"
+  />
 </robot>

File: fingrip_moveit_config/srdf/fingrip_arm.xacro (robot description, xacro)
@@ -7,4 +7,5 @@
   <xacro:macro name="fingrip_arm" params="
     prefix:=fingrip_
+    nbArmjoints:=7
   ">
     <group name="arm">

File: fingrip_moveit_config/srdf/fingrip_gripper.xacro (robot description, xacro)
@@ -5,31 +5,59 @@
   <!-- Macro -->
   <!--       -->
+  <xacro:macro name="noabductionjointtozero" params="
+    prefix:=fingrip_
+    nb_abduction_finger:=2
+    nbFingers:=3
+  ">
+    <xacro:if value="${nbFingers > nb_abduction_finger}">
+        <joint name="${prefix}finger${nbFingers}_proximal_joint" value="0"/>
+        <xacro:noabductionjointtozero
+          prefix="${prefix}"
+          nb_abduction_finger="${nb_abduction_finger}"
+          nbFingers="${nbFingers-1}"
+          />
+    </xacro:if>
+  </xacro:macro>
   <xacro:macro name="fingrip_gripper" params="
     prefix:=fingrip_
+    nbFingers:=3
+    nb_abduction_finger:=2
   ">
     <group name="gripper">
       <link name="${prefix}hand"/>
       <link name="${prefix}palm"/>
-      <link name="${prefix}finger1_base_link"/>
-      <link name="${prefix}finger2_base_link"/>
-      <link name="${prefix}finger3_base_link"/>
-      <joint name="${prefix}finger1_base_joint"/>
-      <joint name="${prefix}finger2_base_joint"/>
+      <xacro:fingrip_gripper_group
+        prefix="${prefix}"
+        nbFingers="$(arg nbFingers)"
+      />
     </group>
-    <group_state name="open" group="gripper">
+    <!-- TODO Depends if abduction there is. -->
+    <group_state name="open_abduction" group="gripper">
       <joint name="${prefix}finger1_base_joint" value="-${pi/2}"/>
       <joint name="${prefix}finger2_base_joint" value="${pi/2}"/>
+      <joint name="${prefix}finger1_proximal_joint" value="0"/>
+      <joint name="${prefix}finger2_proximal_joint" value="0"/>
+      <xacro:noabductionjointtozero
+        prefix="${prefix}"
+        nbFingers="${nbFingers}"
+        nb_abduction_finger="${nb_abduction_finger}"
+      />
     </group_state>
-    <group_state name="close" group="gripper">
+    <group_state name="close_abduction" group="gripper">
       <joint name="${prefix}finger1_base_joint" value="0.0"/>
       <joint name="${prefix}finger2_base_joint" value="0.0"/>
+      <joint name="${prefix}finger1_proximal_joint" value="0"/>
+      <joint name="${prefix}finger2_proximal_joint" value="0"/>
+      <xacro:noabductionjointtozero
+        prefix="${prefix}"
+        nbFingers="${nbFingers}"
+        nb_abduction_finger="${nb_abduction_finger}"
+      />
     </group_state>
     <disable_collisions link1="${prefix}hand" link2="${prefix}palm" reason="Adjacent"/>
-    <disable_collisions link1="${prefix}hand" link2="${prefix}finger1_base_link" reason="Adjacent"/>
-    <disable_collisions link1="${prefix}palm" link2="${prefix}finger1_base_link" reason="Adjacent"/>
-    <disable_collisions link1="${prefix}hand" link2="${prefix}finger2_base_link" reason="Adjacent"/>
-    <disable_collisions link1="${prefix}palm" link2="${prefix}finger2_base_link" reason="Adjacent"/>
-    <disable_collisions link1="${prefix}hand" link2="${prefix}finger3_base_link" reason="Adjacent"/>
-    <disable_collisions link1="${prefix}palm" link2="${prefix}finger3_base_link" reason="Adjacent"/>
+    <xacro:fingrip_gripper_gripper_collision
+        prefix="${prefix}"
+        nbFingers="$(arg nbFingers)"
+    />
     <!-- <disable_collisions link1="${prefix}leftfinger" link2="${prefix}rightfinger" reason="Default"/> -->
   </xacro:macro>

Commit message: MOD: speed of joint fingers and base joint of finger 3 and 4 in passive_joint

File: fingrip_description/urdf/fingrip.urdf (robot description, URDF)
Before this commit: robot fingrip, 19 links, 18 joints
Joints:
- joint fingrip_finger1_base_joint: limit lower=-1.5707963267948966 upper=0 effort=20 velocity=0.2 -> lower=-1.5707963267948966 upper=0 effort=20 velocity=3.14
- joint fingrip_finger2_base_joint: limit lower=0 upper=1.5707963267948966 effort=20 velocity=0.2 -> lower=0 upper=1.5707963267948966 effort=20 velocity=3.14

File: fingrip_description/urdf/fingrip_finger.xacro (robot description, xacro)
@@ -15,5 +15,5 @@
   <xacro:property name="joint_prefix" value="_joint"/>
   <xacro:property name="link_prefix" value="_link"/>
-  <xacro:property name="joint_velocity_limit" value="0.2"/>
+  <xacro:property name="joint_velocity_limit" value="1.57"/> <!-- Before was 0.2 -->
   <xacro:property name="joint_torque_limit" value="20"/>
   <xacro:property name="joint_damping" value="3.0"/>

File: fingrip_moveit_config/srdf/fingrip.srdf.xacro (robot description, xacro)
@@ -36,4 +36,8 @@
     nb_abduction_finger="$(arg nb_abduction_finger)"
   />
+  <group name="arm_gripper">
+    <group name="arm"/>
+    <group name="gripper"/>
+  </group>
   <end_effector group="gripper" name="gripper" parent_group="arm" parent_link="${prefix_arm}hand_tcp"/>
   <!-- Palm And Hand -->

File: fingrip_moveit_config/srdf/fingrip_utils.xacro (robot description, xacro)
@@ -17,7 +17,19 @@
     </xacro:if>
   </xacro:macro>
-  <xacro:macro name="fingrip_gripper_group" params="
+  <xacro:macro name="sub_fingrip_gripper_group_1" params="
     prefix:=fingrip_
     nbFingers:=3
+  ">
+    <xacro:if value="${nbFingers >= 3}">
+      <link name="${prefix}finger${nbFingers}_base_link"/>
+      <link name="${prefix}finger${nbFingers}_proximal_link"/>
+      <passive_joint name="${prefix}finger${nbFingers}_base_joint"/>
+      <joint name="${prefix}finger${nbFingers}_proximal_joint"/>
+      <xacro:sub_fingrip_gripper_group_1 nbFingers="${nbFingers-1}" />
+    </xacro:if>
+  </xacro:macro>
+  <xacro:macro name="sub_fingrip_gripper_group_2" params="
+    prefix:=fingrip_
+    nbFingers:=2
   ">
     <xacro:if value="${nbFingers}">
@@ -26,6 +38,13 @@
       <joint name="${prefix}finger${nbFingers}_base_joint"/>
       <joint name="${prefix}finger${nbFingers}_proximal_joint"/>
-      <xacro:fingrip_gripper_group nbFingers="${nbFingers-1}" />
+      <xacro:sub_fingrip_gripper_group_2 nbFingers="${nbFingers-1}" />
     </xacro:if>
+  </xacro:macro>
+  <xacro:macro name="fingrip_gripper_group" params="
+    prefix:=fingrip_
+    nbFingers:=3
+  ">
+    <xacro:sub_fingrip_gripper_group_1 nbFingers="${nbFingers}"/>
+    <xacro:sub_fingrip_gripper_group_2 nbFingers="2"/>
   </xacro:macro>
   <xacro:macro name="fingrip_gripper_gripper_collision" params="

Commit message: ADD: open gripper and close gripper state

File: fingrip_description/urdf/fingrip.urdf (robot description, URDF)
Before this commit: robot fingrip, 19 links, 18 joints
Joints:
- joint fingrip_finger1_base_joint: limit lower=-1.5707963267948966 upper=0 effort=20 velocity=3.14 -> lower=-1.5707963267948966 upper=0 effort=20 velocity=1.57
- joint fingrip_finger1_proximal_joint: limit lower=-1.3 upper=0.31416 effort=20 velocity=0.2 -> lower=-1.3 upper=0.31416 effort=20 velocity=1.57
- joint fingrip_finger2_base_joint: limit lower=0 upper=1.5707963267948966 effort=20 velocity=3.14 -> lower=0 upper=1.5707963267948966 effort=20 velocity=1.57
- joint fingrip_finger2_proximal_joint: limit lower=-1.3 upper=0.31416 effort=20 velocity=0.2 -> lower=-1.3 upper=0.31416 effort=20 velocity=1.57
- joint fingrip_finger3_proximal_joint: limit lower=-1.3 upper=0.31416 effort=20 velocity=0.2 -> lower=-1.3 upper=0.31416 effort=20 velocity=1.57

File: fingrip_moveit_config/srdf/fingrip_gripper.xacro (robot description, xacro)
@@ -5,18 +5,4 @@
   <!-- Macro -->
   <!--       -->
-  <xacro:macro name="noabductionjointtozero" params="
-    prefix:=fingrip_
-    nb_abduction_finger:=2
-    nbFingers:=3
-  ">
-    <xacro:if value="${nbFingers > nb_abduction_finger}">
-        <joint name="${prefix}finger${nbFingers}_proximal_joint" value="0"/>
-        <xacro:noabductionjointtozero
-          prefix="${prefix}"
-          nb_abduction_finger="${nb_abduction_finger}"
-          nbFingers="${nbFingers-1}"
-          />
-    </xacro:if>
-  </xacro:macro>
   <xacro:macro name="fingrip_gripper" params="
     prefix:=fingrip_
@@ -36,22 +22,21 @@
       <joint name="${prefix}finger1_base_joint" value="-${pi/2}"/>
       <joint name="${prefix}finger2_base_joint" value="${pi/2}"/>
-      <joint name="${prefix}finger1_proximal_joint" value="0"/>
-      <joint name="${prefix}finger2_proximal_joint" value="0"/>
-      <xacro:noabductionjointtozero
-        prefix="${prefix}"
-        nbFingers="${nbFingers}"
-        nb_abduction_finger="${nb_abduction_finger}"
-      />
     </group_state>
     <group_state name="close_abduction" group="gripper">
       <joint name="${prefix}finger1_base_joint" value="0.0"/>
       <joint name="${prefix}finger2_base_joint" value="0.0"/>
-      <joint name="${prefix}finger1_proximal_joint" value="0"/>
-      <joint name="${prefix}finger2_proximal_joint" value="0"/>
-      <xacro:noabductionjointtozero
-        prefix="${prefix}"
-        nbFingers="${nbFingers}"
-        nb_abduction_finger="${nb_abduction_finger}"
-      />
+    </group_state>
+    <!-- ADD dependencies if there are more fingers -->
+    <!-- The closing or opening of the proximal joint should have an impact onto the intermediaire and distal
+     through under-actuated joints -->
+    <group_state name="close" group="gripper">
+      <joint name="${prefix}finger1_proximal_joint" value="${18*pi/180}"/>
+      <joint name="${prefix}finger2_proximal_joint" value="${18*pi/180}"/>
+      <joint name="${prefix}finger3_proximal_joint" value="${18*pi/180}"/>
+    </group_state>
+    <group_state name="open" group="gripper">
+      <joint name="${prefix}finger1_proximal_joint" value="-${74*pi/180}"/>
+      <joint name="${prefix}finger2_proximal_joint" value="-${74*pi/180}"/>
+      <joint name="${prefix}finger3_proximal_joint" value="-${74*pi/180}"/>
     </group_state>
     <disable_collisions link1="${prefix}hand" link2="${prefix}palm" reason="Adjacent"/>
