Commit message: ADD: intermediaire joints

File: fingrip_description/urdf/fingrip.urdf (robot description, URDF)
Before this commit: robot fingrip, 19 links, 18 joints
Links:
- added link fingrip_finger1_intermediaire_link, mass 0.150; collision mesh filename=package://fingrip_description/meshes/collision/gripper/inte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; visual mesh filename=package://fingrip_description/meshes/visual/gripper/interme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
- added link fingrip_finger2_intermediaire_link, mass 0.150; collision mesh filename=package://fingrip_description/meshes/collision/gripper/inte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; visual mesh filename=package://fingrip_description/meshes/visual/gripper/interme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
- added link fingrip_finger3_intermediaire_link, mass 0.150; collision mesh filename=package://fingrip_description/meshes/collision/gripper/inte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; visual mesh filename=package://fingrip_description/meshes/visual/gripper/interme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
- link fingrip_finger1_proximal_link: mass 0.2238453537819424 -> 0.150
- link fingrip_finger2_proximal_link: mass 0.2238453537819424 -> 0.150
- link fingrip_finger3_proximal_link: mass 0.2238453537819424 -> 0.150
Joints:
- added joint fingrip_finger1_intermediaire_joint: type revolute, parent fingrip_finger1_proximal_link, child fingrip_finger1_intermediaire_link, origin xyz=0.08 0 0 rpy=0 0 0, axis 0 0 1, limit lower=-0.5 upper=1.0472 effort=20 velocity=1.57
- added joint fingrip_finger2_intermediaire_joint: type revolute, parent fingrip_finger2_proximal_link, child fingrip_finger2_intermediaire_link, origin xyz=0.08 0 0 rpy=0 0 0, axis 0 0 1, limit lower=-0.5 upper=1.0472 effort=20 velocity=1.57
- added joint fingrip_finger3_intermediaire_joint: type revolute, parent fingrip_finger3_proximal_link, child fingrip_finger3_intermediaire_link, origin xyz=0.08 0 0 rpy=0 0 0, axis 0 0 1, limit lower=-0.5 upper=1.0472 effort=20 velocity=1.57

File: fingrip_description/urdf/fingrip_finger.xacro (robot description, xacro)
@@ -34,5 +34,5 @@
   <xacro:property name="joint_intermediaire_lower_limit" value="-0.5"/>
   <xacro:property name="joint_intermediaire_upper_limit" value="1.0472"/>
-  <xacro:property name="joint_intermediaire_origin_xyz" value="0 0 0.0584"/>
+  <xacro:property name="joint_intermediaire_origin_xyz" value="0.08 0 0"/>
   <xacro:property name="joint_intermediaire_origin_rpy" value="0 0 0"/>
   <xacro:property name="joint_intermediaire_axis_xyz" value="0 0 1"/>
@@ -112,5 +112,4 @@
         />
         <!-- INTERMEDIAIRE limb -->
-        <!--
         <xacro:fingrip_joint
         parent="${prefix}${finger_name}${proximal_prefix}${link_prefix}"
@@ -118,9 +117,9 @@
         joint_name="${prefix}${finger_name}${intermediaire_prefix}${joint_prefix}"
         joint_type="${joint_other_type}"
-        joint_origin_xyz="${joint_other_origin_xyz}"
-        joint_origin_rpy="${joint_other_origin_rpy}"
-        joint_axis_xyz="${joint_other_axis_xyz}"
-        joint_lower_limit="${joint_lower_limit}"
-        joint_upper_limit="${joint_upper_limit}"
+        joint_origin_xyz="${joint_intermediaire_origin_xyz}"
+        joint_origin_rpy="${joint_intermediaire_origin_rpy}"
+        joint_axis_xyz="${joint_intermediaire_axis_xyz}"
+        joint_lower_limit="${joint_intermediaire_lower_limit}"
+        joint_upper_limit="${joint_intermediaire_upper_limit}"
         joint_velocity_limit="${joint_velocity_limit}"
         joint_torque_limit="${joint_torque_limit}"
@@ -135,5 +134,4 @@
         mu="${link_mu}"
         />
-        -->
         <!-- DISTAL limb -->
         <!--

File: fingrip_description/urdf/fingrip_inertial.xacro (robot description, xacro)
@@ -142,5 +142,5 @@
       <inertial>
         <origin xyz="0.03411 -0.01012 0.0" rpy="${mesh_offset_rpy}"/>
-        <mass value="0.2238453537819424"/>
+        <mass value="0.150"/>
         <inertia ixx="0.000092" ixy="-0.000061" ixz="0.0" iyy="0.00031" iyz="0.0" izz="0.00031"/>
       </inertial>
@@ -150,5 +150,5 @@
       <inertial>
         <origin xyz="0.01791 -0.01023 0.0" rpy="${mesh_offset_rpy}"/>
-        <mass value="0.2238453537819424"/>
+        <mass value="0.150"/>
         <inertia ixx="0.000025" ixy="0.000013" ixz="0.0" iyy="0.000102" iyz="0.0" izz="0.000108"/>
       </inertial>
@@ -158,5 +158,5 @@
       <inertial>
         <origin xyz="0.01217 -0.00732 0.0" rpy="${mesh_offset_rpy}"/>
-        <mass value="0.2238453537819424"/>
+        <mass value="0.1"/>
         <inertia ixx="0.000025" ixy="0.000013" ixz="0.0" iyy="0.000102" iyz="0.0" izz="0.000108"/>
       </inertial>

File: fingrip_moveit_config/srdf/fingrip_gripper.xacro (robot description, xacro)
@@ -41,5 +41,9 @@
     </group_state>
     <disable_collisions link1="${prefix}hand" link2="${prefix}palm" reason="Adjacent"/>
-    <xacro:fingrip_gripper_gripper_collision
+    <xacro:fingrip_gripper_base_collision
+        prefix="${prefix}"
+        nbFingers="$(arg nbFingers)"
+    />
+    <xacro:fingrip_gripper_finger_collision
         prefix="${prefix}"
         nbFingers="$(arg nbFingers)"

File: fingrip_moveit_config/srdf/fingrip_utils.xacro (robot description, xacro)
@@ -2,4 +2,13 @@
 <!-- Macro for SRDF of Franka Emika fingrip arm -->
 <robot xmlns:xacro="http://wiki.ros.org/xacro">
+  <!--            -->
+  <!-- Properties -->
+  <!-- GENERAL    -->
+  <xacro:property name="base_prefix" value="_base"/>
+  <xacro:property name="proximal_prefix" value="_proximal"/>
+  <xacro:property name="intermediaire_prefix" value="_intermediaire"/>
+  <xacro:property name="distal_prefix" value="_distal"/>
+  <xacro:property name="joint_prefix" value="_joint"/>
+  <xacro:property name="link_prefix" value="_link"/>
   <!--       -->
   <!-- Macro -->
@@ -11,7 +20,7 @@
   ">
     <xacro:if value="${nbFingers}">
-        <disable_collisions link1="${prefix_gripper}finger${nbFingers}_base_link" link2="${prefix_arm}link3" reason="Never"/>
-        <disable_collisions link1="${prefix_gripper}finger${nbFingers}_base_link" link2="${prefix_arm}link4" reason="Never"/>
-        <disable_collisions link1="${prefix_gripper}finger${nbFingers}_base_link" link2="${prefix_arm}link6" reason="Never"/>
+        <disable_collisions link1="${prefix_gripper}finger${nbFingers}${base_prefix}${link_prefix}" link2="${prefix_arm}link3" reason="Never"/>
+        <disable_collisions link1="${prefix_gripper}finger${nbFingers}${base_prefix}${link_prefix}" link2="${prefix_arm}link4" reason="Never"/>
+        <disable_collisions link1="${prefix_gripper}finger${nbFingers}${base_prefix}${link_prefix}" link2="${prefix_arm}link6" reason="Never"/>
         <xacro:fingrip_gripper_arm_collision nbFingers="${nbFingers-1}" />
     </xacro:if>
@@ -22,8 +31,10 @@
   ">
     <xacro:if value="${nbFingers >= 3}">
-      <link name="${prefix}finger${nbFingers}_base_link"/>
-      <link name="${prefix}finger${nbFingers}_proximal_link"/>
-      <passive_joint name="${prefix}finger${nbFingers}_base_joint"/>
-      <joint name="${prefix}finger${nbFingers}_proximal_joint"/>
+      <link name="${prefix}finger${nbFingers}${base_prefix}${link_prefix}"/>
+      <link name="${prefix}finger${nbFingers}${proximal_prefix}${link_prefix}"/>
+      <link name="${prefix}finger${nbFingers}${intermediaire_prefix}${link_prefix}"/>
+      <passive_joint name="${prefix}finger${nbFingers}${base_prefix}${joint_prefix}"/>
+      <joint name="${prefix}finger${nbFingers}${proximal_prefix}${joint_prefix}"/>
+      <joint name="${prefix}finger${nbFingers}${intermediaire_prefix}${joint_prefix}"/>
       <xacro:sub_fingrip_gripper_group_1 nbFingers="${nbFingers-1}" />
     </xacro:if>
@@ -34,8 +45,10 @@
   ">
     <xacro:if value="${nbFingers}">
-      <link name="${prefix}finger${nbFingers}_base_link"/>
-      <link name="${prefix}finger${nbFingers}_proximal_link"/>
-      <joint name="${prefix}finger${nbFingers}_base_joint"/>
-      <joint name="${prefix}finger${nbFingers}_proximal_joint"/>
+      <link name="${prefix}finger${nbFingers}${base_prefix}${link_prefix}"/>
+      <link name="${prefix}finger${nbFingers}${proximal_prefix}${link_prefix}"/>
+      <link name="${prefix}finger${nbFingers}${intermediaire_prefix}${link_prefix}"/>
+      <joint name="${prefix}finger${nbFingers}${base_prefix}${joint_prefix}"/>
+      <joint name="${prefix}finger${nbFingers}${proximal_prefix}${joint_prefix}"/>
+      <joint name="${prefix}finger${nbFingers}${intermediaire_prefix}${joint_prefix}"/>
       <xacro:sub_fingrip_gripper_group_2 nbFingers="${nbFingers-1}" />
     </xacro:if>
@@ -48,12 +61,22 @@
     <xacro:sub_fingrip_gripper_group_2 nbFingers="2"/>
   </xacro:macro>
-  <xacro:macro name="fingrip_gripper_gripper_collision" params="
+  <xacro:macro name="fingrip_gripper_base_collision" params="
     prefix:=fingrip_
     nbFingers:=3
   ">
     <xacro:if value="${nbFingers}">
-        <disable_collisions link1="${prefix}hand" link2="${prefix}finger${nbFingers}_base_link" reason="Adjacent"/>
-        <disable_collisions link1="${prefix}palm" link2="${prefix}finger${nbFingers}_base_link" reason="Adjacent"/>
-        <xacro:fingrip_gripper_gripper_collision nbFingers="${nbFingers-1}" />
+        <disable_collisions link1="${prefix}hand" link2="${prefix}finger${nbFingers}${base_prefix}${link_prefix}" reason="Adjacent"/>
+        <disable_collisions link1="${prefix}palm" link2="${prefix}finger${nbFingers}${base_prefix}${link_prefix}" reason="Adjacent"/>
+        <xacro:fingrip_gripper_base_collision nbFingers="${nbFingers-1}" />
+    </xacro:if>
+  </xacro:macro>
+  <xacro:macro name="fingrip_gripper_finger_collision" params="
+    prefix:=fingrip_
+    nbFingers:=3
+  ">
+    <xacro:if value="${nbFingers}">
+        <disable_collisions link1="${prefix}finger${nbFingers}${base_prefix}${link_prefix}" link2="${prefix}finger${nbFingers}${proximal_prefix}${link_prefix}" reason="Adjacent"/>
+        <disable_collisions link1="${prefix}finger${nbFingers}${proximal_prefix}${link_prefix}" link2="${prefix}finger${nbFingers}${intermediaire_prefix}${link_prefix}" reason="Adjacent"/>
+        <xacro:fingrip_gripper_finger_collision nbFingers="${nbFingers-1}" />
     </xacro:if>
   </xacro:macro>
