Commit message: ADD: change panda arm to Kuka (OK), (WIP) change the gripper

File: fingrip_description/urdf/fingrip.urdf.xacro (robot description, xacro)
@@ -2,4 +2,5 @@
 <!-- URDF for Franka Emika fingrip -->
 <robot xmlns:xacro="http://wiki.ros.org/xacro" name="$(arg name)">
+  <!-- NEW ONE AGAIN -->
   <!--                   -->
   <!-- Imported elements -->
@@ -40,4 +41,12 @@
   <!-- Flag to preserve fixed joints and prevent lumping when generating SDF for Gazebo -->
   <xacro:arg name="gazebo_preserve_fixed_joint" default="false"/>
+  <!-- Flag to use 3 or 4 fingers model  -->
+  <xacro:arg name="underactuation" default="true"/>
+  <!-- Flag to use underactuation model -->
+  <xacro:arg name="longFingertip" default="false"/>
+  <!-- Flag to use long or short fingers model  -->
+  <xacro:arg name="nbFingers" default="3"/>
+  <!-- Flag to use small or bigger palm size  -->
+  <xacro:arg name="hand_type" default="1"/>
   <!--            -->
   <!-- Properties -->
@@ -53,4 +62,14 @@
   <xacro:property name="gripper_offset_xyz" value="0 0 0"/>
   <xacro:property name="gripper_offset_rpy" value="0 0 0"/>
+  <!-- Import Rviz colors -->
+  <material name="Grey">
+    <color rgba="0.2 0.2 0.2 1.0"/>
+  </material>
+  <material name="Orange">
+    <color rgba="1.0 0.423529411765 0.0392156862745 1.0"/>
+  </material>
+  <material name="Blue">
+    <color rgba="0.5 0.7 1.0 1.0"/>
+  </material>
   <!--       -->
   <!-- Robot -->
@@ -89,4 +108,8 @@
       ros2_control_command_interface="$(arg ros2_control_command_interface)"
       gazebo_preserve_fixed_joint="$(arg gazebo_preserve_fixed_joint)"
+      underactuation="$(arg underactuation)"
+      longFingertip="$(arg longFingertip)"
+      nbFingers="$(arg nbFingers)"
+      hand_type="$(arg hand_type)"
     />
   </xacro:if>

File: fingrip_description/urdf/fingrip_arm.xacro (robot description, xacro)
@@ -14,12 +14,13 @@
   <xacro:property name="link0_name" value="link0"/>
   <xacro:property name="link0_mu" value="0.85"/>
+  <xacro:property name="link0_color" value="Grey"/>
   <xacro:property name="joint1_name" value="joint1"/>
   <xacro:property name="joint1_type" value="revolute"/>
-  <xacro:property name="joint1_origin_xyz" value="0 0 0.333"/>
+  <xacro:property name="joint1_origin_xyz" value="0 0 0.1575"/>
   <xacro:property name="joint1_origin_rpy" value="0 0 0"/>
   <xacro:property name="joint1_axis_xyz" value="0 0 1"/>
-  <xacro:property name="joint1_lower_limit" value="${-166*pi/180}"/>
-  <xacro:property name="joint1_upper_limit" value="${166*pi/180}"/>
-  <xacro:property name="joint1_velocity_limit" value="${150*pi/180}"/>
+  <xacro:property name="joint1_lower_limit" value="${-170*pi/180}"/>
+  <xacro:property name="joint1_upper_limit" value="${170*pi/180}"/>
+  <xacro:property name="joint1_velocity_limit" value="${85*pi/180}"/>
   <xacro:property name="joint1_torque_limit" value="87"/>
   <xacro:property name="joint1_damping" value="21.75"/>
@@ -27,12 +28,13 @@
   <xacro:property name="link1_name" value="link1"/>
   <xacro:property name="link1_mu" value="0.85"/>
+  <xacro:property name="link1_color" value="Blue"/>
   <xacro:property name="joint2_name" value="joint2"/>
   <xacro:property name="joint2_type" value="revolute"/>
-  <xacro:property name="joint2_origin_xyz" value="0 0 0"/>
-  <xacro:property name="joint2_origin_rpy" value="${-pi/2} 0 0"/>
+  <xacro:property name="joint2_origin_xyz" value="0 0 0.2025"/>
+  <xacro:property name="joint2_origin_rpy" value="${pi/2} 0 ${-pi}"/>
   <xacro:property name="joint2_axis_xyz" value="0 0 1"/>
-  <xacro:property name="joint2_lower_limit" value="${-101*pi/180}"/>
-  <xacro:property name="joint2_upper_limit" value="${101*pi/180}"/>
-  <xacro:property name="joint2_velocity_limit" value="${150*pi/180}"/>
+  <xacro:property name="joint2_lower_limit" value="${-120*pi/180}"/>
+  <xacro:property name="joint2_upper_limit" value="${120*pi/180}"/>
+  <xacro:property name="joint2_velocity_limit" value="${85*pi/180}"/>
   <xacro:property name="joint2_torque_limit" value="87"/>
   <xacro:property name="joint2_damping" value="21.75"/>
@@ -40,12 +42,13 @@
   <xacro:property name="link2_name" value="link2"/>
   <xacro:property name="link2_mu" value="0.85"/>
+  <xacro:property name="link2_color" value="Blue"/>
   <xacro:property name="joint3_name" value="joint3"/>
   <xacro:property name="joint3_type" value="revolute"/>
-  <xacro:property name="joint3_origin_xyz" value="0 -0.316 0"/>
-  <xacro:property name="joint3_origin_rpy" value="${pi/2} 0 0"/>
+  <xacro:property name="joint3_origin_xyz" value="0 0.2045 0"/>
+  <xacro:property name="joint3_origin_rpy" value="${pi/2} 0 ${-pi}"/>
   <xacro:property name="joint3_axis_xyz" value="0 0 1"/>
-  <xacro:property name="joint3_lower_limit" value="${-166*pi/180}"/>
-  <xacro:property name="joint3_upper_limit" value="${166*pi/180}"/>
-  <xacro:property name="joint3_velocity_limit" value="${150*pi/180}"/>
+  <xacro:property name="joint3_lower_limit" value="${-170*pi/180}"/>
+  <xacro:property name="joint3_upper_limit" value="${170*pi/180}"/>
+  <xacro:property name="joint3_velocity_limit" value="${100*pi/180}"/>
   <xacro:property name="joint3_torque_limit" value="87"/>
   <xacro:property name="joint3_damping" value="21.75"/>
@@ -53,12 +56,13 @@
   <xacro:property name="link3_name" value="link3"/>
   <xacro:property name="link3_mu" value="0.85"/>
+  <xacro:property name="link3_color" value="Orange"/>
   <xacro:property name="joint4_name" value="joint4"/>
   <xacro:property name="joint4_type" value="revolute"/>
-  <xacro:property name="joint4_origin_xyz" value="0.0825 0 0"/>
+  <xacro:property name="joint4_origin_xyz" value="0.0 0.0 0.2155"/>
   <xacro:property name="joint4_origin_rpy" value="${pi/2} 0 0"/>
   <xacro:property name="joint4_axis_xyz" value="0 0 1"/>
-  <xacro:property name="joint4_lower_limit" value="${-176/180*pi}"/>
-  <xacro:property name="joint4_upper_limit" value="${-4/180*pi}"/>
-  <xacro:property name="joint4_velocity_limit" value="${150*pi/180}"/>
+  <xacro:property name="joint4_lower_limit" value="${-120/180*pi}"/>
+  <xacro:property name="joint4_upper_limit" value="${120/180*pi}"/>
+  <xacro:property name="joint4_velocity_limit" value="${75*pi/180}"/>
   <xacro:property name="joint4_torque_limit" value="87"/>
   <xacro:property name="joint4_damping" value="21.75"/>
@@ -66,12 +70,13 @@
   <xacro:property name="link4_name" value="link4"/>
   <xacro:property name="link4_mu" value="0.85"/>
+  <xacro:property name="link4_color" value="Blue"/>
   <xacro:property name="joint5_name" value="joint5"/>
   <xacro:property name="joint5_type" value="revolute"/>
-  <xacro:property name="joint5_origin_xyz" value="-0.0825 0.384 0"/>
-  <xacro:property name="joint5_origin_rpy" value="${-pi/2} 0 0"/>
+  <xacro:property name="joint5_origin_xyz" value="0.0 0.1845 0.0"/>
+  <xacro:property name="joint5_origin_rpy" value="${pi/2} 0 ${pi}"/>
   <xacro:property name="joint5_axis_xyz" value="0 0 1"/>
-  <xacro:property name="joint5_lower_limit" value="${-166*pi/180}"/>
-  <xacro:property name="joint5_upper_limit" value="${166*pi/180}"/>
-  <xacro:property name="joint5_velocity_limit" value="${pi}"/>
+  <xacro:property name="joint5_lower_limit" value="${-170*pi/180}"/>
+  <xacro:property name="joint5_upper_limit" value="${170*pi/180}"/>
+  <xacro:property name="joint5_velocity_limit" value="${130*pi/180}"/>
   <xacro:property name="joint5_torque_limit" value="12"/>
   <xacro:property name="joint5_damping" value="3.0"/>
@@ -79,12 +84,13 @@
   <xacro:property name="link5_name" value="link5"/>
   <xacro:property name="link5_mu" value="0.85"/>
+  <xacro:property name="link5_color" value="Blue"/>
   <xacro:property name="joint6_name" value="joint6"/>
   <xacro:property name="joint6_type" value="revolute"/>
-  <xacro:property name="joint6_origin_xyz" value="0 0 0"/>
+  <xacro:property name="joint6_origin_xyz" value="0.0 0.0 0.2155"/>
   <xacro:property name="joint6_origin_rpy" value="${pi/2} 0 0"/>
   <xacro:property name="joint6_axis_xyz" value="0 0 1"/>
-  <xacro:property name="joint6_lower_limit" value="${-1/180*pi}"/>
-  <xacro:property name="joint6_upper_limit" value="${215/180*pi}"/>
-  <xacro:property name="joint6_velocity_limit" value="${pi}"/>
+  <xacro:property name="joint6_lower_limit" value="${-120/180*pi}"/>
+  <xacro:property name="joint6_upper_limit" value="${120/180*pi}"/>
+  <xacro:property name="joint6_velocity_limit" value="${135*pi/180}"/>
   <xacro:property name="joint6_torque_limit" value="12"/>
   <xacro:property name="joint6_damping" value="3.0"/>
@@ -92,12 +98,13 @@
   <xacro:property name="link6_name" value="link6"/>
   <xacro:property name="link6_mu" value="0.85"/>
+  <xacro:property name="link6_color" value="Orange"/>
   <xacro:property name="joint7_name" value="joint7"/>
   <xacro:property name="joint7_type" value="revolute"/>
-  <xacro:property name="joint7_origin_xyz" value="0.088 0 0"/>
-  <xacro:property name="joint7_origin_rpy" value="${pi/2} 0 0"/>
+  <xacro:property name="joint7_origin_xyz" value="0.0 0.081 0.0"/>
+  <xacro:property name="joint7_origin_rpy" value="${pi/2} 0 ${-pi}"/>
   <xacro:property name="joint7_axis_xyz" value="0 0 1"/>
-  <xacro:property name="joint7_lower_limit" value="${-166*pi/180}"/>
-  <xacro:property name="joint7_upper_limit" value="${166*pi/180}"/>
-  <xacro:property name="joint7_velocity_limit" value="${pi}"/>
+  <xacro:property name="joint7_lower_limit" value="${-175*pi/180}"/>
+  <xacro:property name="joint7_upper_limit" value="${175*pi/180}"/>
+  <xacro:property name="joint7_velocity_limit" value="${135*pi/180}"/>
   <xacro:property name="joint7_torque_limit" value="12"/>
   <xacro:property name="joint7_damping" value="3.0"/>
@@ -105,4 +112,5 @@
   <xacro:property name="link7_name" value="link7"/>
   <xacro:property name="link7_mu" value="0.85"/>
+  <xacro:property name="link7_color" value="Grey"/>
   <xacro:property name="wrist_flange_name" value="link8"/>
   <xacro:property name="wrist_flange_origin_xyz" value="0 0 0.107"/>
@@ -143,4 +151,5 @@
     collision="${collision}"
     mu="${link0_mu}"
+    color="${link0_color}"
     />
     <!-- 1 -->
@@ -170,4 +179,5 @@
     collision="${collision}"
     mu="${link1_mu}"
+    color="${link1_color}"
     />
     <!-- 2 -->
@@ -197,4 +207,5 @@
     collision="${collision}"
     mu="${link2_mu}"
+    color="${link2_color}"
     />
     <!-- 3 -->
@@ -224,4 +235,5 @@
     collision="${collision}"
     mu="${link3_mu}"
+    color="${link3_color}"
     />
     <!-- 4 -->
@@ -251,4 +263,5 @@
     collision="${collision}"
     mu="${link4_mu}"
+    color="${link4_color}"
     />
     <!-- 5 -->
@@ -278,4 +291,5 @@
     collision="${collision}"
     mu="${link5_mu}"
+    color="${link5_color}"
     />
     <!-- 6 -->
@@ -305,4 +319,5 @@
     collision="${collision}"
     mu="${link6_mu}"
+    color="${link6_color}"
     />
     <!-- 7 -->
@@ -332,4 +347,5 @@
     collision="${collision}"
     mu="${link7_mu}"
+    color="${link7_color}"
     />
     <!-- Wrist flange -->

File: fingrip_description/urdf/fingrip_gripper.xacro (robot description, xacro)
@@ -5,44 +5,44 @@
   <!-- Imported elements -->
   <!--                   -->
-  <xacro:include filename="$(find fingrip_description)/urdf/fingrip_utils.xacro"/>
   <xacro:include filename="$(find fingrip_description)/urdf/fingrip.ros2_control"/>
+  <xacro:include filename="$(find fingrip_description)/urdf/fingrip_finger.xacro"/>
+  <xacro:include filename="$(find fingrip_description)/urdf/fingrip_palm.xacro"/>
   <!--            -->
   <!-- Properties -->
   <!--            -->
+  <!-- WRIST -->
   <xacro:property name="joint_wrist_name" value="joint_wrist"/>
   <xacro:property name="joint_wrist_type" value="fixed"/>
   <xacro:property name="hand_name" value="hand"/>
   <xacro:property name="hand_mu" value="0.85"/>
-  <xacro:property name="joint_finger1_name" value="finger_joint1"/>
-  <xacro:property name="joint_finger1_type" value="prismatic"/>
-  <xacro:property name="joint_finger1_origin_xyz" value="0 0 0.0584"/>
-  <xacro:property name="joint_finger1_origin_rpy" value="0 0 0"/>
-  <xacro:property name="joint_finger1_axis_xyz" value="0 1 0"/>
-  <xacro:property name="joint_finger1_lower_limit" value="0"/>
-  <xacro:property name="joint_finger1_upper_limit" value="0.04"/>
-  <xacro:property name="joint_finger1_velocity_limit" value="0.2"/>
-  <xacro:property name="joint_finger1_torque_limit" value="20"/>
-  <xacro:property name="joint_finger1_damping" value="3.0"/>
-  <xacro:property name="joint_finger1_friction" value="0.4"/>
-  <xacro:property name="link_finger1_name" value="leftfinger"/>
-  <xacro:property name="link_finger1_mu" value="1.13"/>
+  <!-- Finger dependent properties -->
+  <!-- FINGER 1 -->
+  <xacro:property name="finger1_name" value="finger1"/>
+  <xacro:property name="joint_finger1_base_type" value="revolute"/>
+  <xacro:property name="joint_finger1_base_origin_xyz" value="0 0 0.0584"/>
+  <xacro:property name="joint_finger1_base_origin_rpy" value="0 0 0"/>
+  <xacro:property name="joint_finger1_base_axis_xyz" value="0 1 0"/>
   <xacro:property name="link_finger1_mesh_offset" value="0 0 0"/>
-  <xacro:property name="joint_finger2_name" value="finger_joint2"/>
-  <xacro:property name="joint_finger2_type" value="prismatic"/>
-  <xacro:property name="joint_finger2_origin_xyz" value="0 0 0.0584"/>
-  <xacro:property name="joint_finger2_origin_rpy" value="0 0 0"/>
-  <xacro:property name="joint_finger2_axis_xyz" value="0 -1 0"/>
-  <xacro:property name="joint_finger2_lower_limit" value="0"/>
-  <xacro:property name="joint_finger2_upper_limit" value="0.04"/>
-  <xacro:property name="joint_finger2_velocity_limit" value="0.2"/>
-  <xacro:property name="joint_finger2_torque_limit" value="20"/>
-  <xacro:property name="joint_finger2_damping" value="3.0"/>
-  <xacro:property name="joint_finger2_friction" value="0.4"/>
-  <xacro:property name="link_finger2_name" value="rightfinger"/>
-  <xacro:property name="link_finger2_mu" value="1.13"/>
-  <xacro:property name="link_finger2_mesh_offset" value="0 0 ${pi}"/>
-  <xacro:property name="ee_name" value="hand_tcp"/>
-  <xacro:property name="ee_origin_xyz" value="0 0 0.1034"/>
-  <xacro:property name="ee_origin_rpy" value="0 0 0"/>
+  <!-- FINGER 2 -->
+  <xacro:property name="finger2_name" value="finger2"/>
+  <xacro:property name="joint_finger2_base_type" value="revolute"/>
+  <xacro:property name="joint_finger2_base_origin_xyz" value="0 0 0.0584"/>
+  <xacro:property name="joint_finger2_base_origin_rpy" value="0 0 0"/>
+  <xacro:property name="joint_finger2_base_axis_xyz" value="0 1 0"/>
+  <xacro:property name="link_finger2_mesh_offset" value="0 0 0"/>
+  <!-- FINGER 3 -->
+  <xacro:property name="finger3_name" value="finger3"/>
+  <xacro:property name="joint_finger3_base_type" value="fixed"/>
+  <xacro:property name="joint_finger3_base_origin_xyz" value="0 0 0.0584"/>
+  <xacro:property name="joint_finger3_base_origin_rpy" value="0 0 0"/>
+  <xacro:property name="joint_finger3_base_axis_xyz" value="0 1 0"/>
+  <xacro:property name="link_finger3_mesh_offset" value="0 0 0"/>
+  <!-- FINGER 4 -->
+  <xacro:property name="finger4_name" value="finger4"/>
+  <xacro:property name="joint_finger4_base_type" value="fixed"/>
+  <xacro:property name="joint_finger4_base_origin_xyz" value="0 0 0.0584"/>
+  <xacro:property name="joint_finger4_base_origin_rpy" value="0 0 0"/>
+  <xacro:property name="joint_finger4_base_axis_xyz" value="0 1 0"/>
+  <xacro:property name="link_finger4_mesh_offset" value="0 0 0"/>
   <!--       -->
   <!-- Macro -->
@@ -60,69 +60,78 @@
     ros2_control_command_interface:=effort
     gazebo_preserve_fixed_joint:=false
+    underactuation:=true
+    longFingertip:=false
+    nbFingers:=3
+    hand_type:=1
   ">
-    <!-- Wrist -->
-    <xacro:fingrip_joint
-    parent="${wrist_flange}"
-    child="${prefix}${hand_name}"
-    joint_name="${prefix}${joint_wrist_name}"
-    joint_type="${joint_wrist_type}"
-    joint_origin_xyz="${origin_xyz}"
-    joint_origin_rpy="${origin_rpy}"
-    gazebo_preserve_fixed_joint="${gazebo_preserve_fixed_joint}"
-    />
-    <xacro:fingrip_link
-    link_name="${prefix}${hand_name}"
-    mesh="${hand_mesh}"
-    collision="${collision}"
-    mu="${hand_mu}"
-    />
-    <!-- Finger 1 -->
-    <xacro:fingrip_joint
-    parent="${prefix}${hand_name}"
-    child="${prefix}${link_finger1_name}"
-    joint_name="${prefix}${joint_finger1_name}"
-    joint_type="${joint_finger1_type}"
-    joint_origin_xyz="${joint_finger1_origin_xyz}"
-    joint_origin_rpy="${joint_finger1_origin_rpy}"
-    joint_axis_xyz="${joint_finger1_axis_xyz}"
-    joint_lower_limit="${joint_finger1_lower_limit}"
-    joint_upper_limit="${joint_finger1_upper_limit}"
-    joint_velocity_limit="${joint_finger1_velocity_limit}"
-    joint_torque_limit="${joint_finger1_torque_limit}"
-    joint_damping="${joint_finger1_damping}"
-    joint_friction="${joint_finger1_friction}"
-    gazebo_preserve_fixed_joint="${gazebo_preserve_fixed_joint}"
-    />
-    <xacro:fingrip_link
-    link_name="${prefix}${link_finger1_name}"
-    mesh="${finger_mesh}"
-    collision="${collision}"
-    mu="${link_finger1_mu}"
-    mesh_offset_rpy="${link_finger1_mesh_offset}"
-    />
-    <!-- Finger 2 -->
-    <xacro:fingrip_joint
-    parent="${prefix}${hand_name}"
-    child="${prefix}${link_finger2_name}"
-    joint_name="${prefix}${joint_finger2_name}"
-    joint_type="${joint_finger2_type}"
-    joint_origin_xyz="${joint_finger2_origin_xyz}"
-    joint_origin_rpy="${joint_finger2_origin_rpy}"
-    joint_axis_xyz="${joint_finger2_axis_xyz}"
-    joint_lower_limit="${joint_finger2_lower_limit}"
-    joint_upper_limit="${joint_finger2_upper_limit}"
-    joint_velocity_limit="${joint_finger2_velocity_limit}"
-    joint_torque_limit="${joint_finger2_torque_limit}"
-    joint_damping="${joint_finger2_damping}"
-    joint_friction="${joint_finger2_friction}"
-    gazebo_preserve_fixed_joint="${gazebo_preserve_fixed_joint}"
-    />
-    <xacro:fingrip_link
-    link_name="${prefix}${link_finger2_name}"
-    mesh="${finger_mesh}"
-    collision="${collision}"
-    mu="${link_finger2_mu}"
-    mesh_offset_rpy="${link_finger2_mesh_offset}"
-    />
+        <!-- Wrist & Palm -->
+        <xacro:fingrip_palm
+        parent="${wrist_flange}"
+        prefix="${prefix}"
+        hand_name="${hand_name}"
+        joint_name="${prefix}${joint_wrist_name}"
+        joint_type="${joint_wrist_type}"
+        joint_origin_xyz="${origin_xyz}"
+        joint_origin_rpy="${origin_rpy}"
+        gazebo_preserve_fixed_joint="${gazebo_preserve_fixed_joint}"
+        collision="${collision}"
+        mu="${hand_mu}"
+        nbFingers="${nbFingers}"
+        handtype="${hand_type}"
+        />
+        <!-- Finger 1 -->
+        <xacro:fingrip_finger
+        finger_name="${finger1_name}"
+        collision="${collision}"
+        mesh_offset_rpy="${link_finger1_mesh_offset}"
+        parent="${prefix}${hand_name}"
+        prefix="${prefix}"
+        joint_type="${joint_finger1_base_type}"
+        joint_origin_xyz="${joint_finger1_base_origin_xyz}"
+        joint_origin_rpy="${joint_finger1_base_origin_rpy}"
+        joint_axis_xyz="${joint_finger1_base_axis_xyz}"
+        gazebo_preserve_fixed_joint="${gazebo_preserve_fixed_joint}"
+        />
+        <!-- FINGER 2 -->
+        <xacro:fingrip_finger
+        finger_name="${finger2_name}"
+        collision="${collision}"
+        mesh_offset_rpy="${link_finger2_mesh_offset}"
+        parent="${prefix}${hand_name}"
+        prefix="${prefix}"
+        joint_type="${joint_finger2_base_type}"
+        joint_origin_xyz="${joint_finger2_base_origin_xyz}"
+        joint_origin_rpy="${joint_finger2_base_origin_rpy}"
+        joint_axis_xyz="${joint_finger2_base_axis_xyz}"
+        gazebo_preserve_fixed_joint="${gazebo_preserve_fixed_joint}"
+        />
+        <!-- FINGER 3 -->
+        <xacro:fingrip_finger
+        finger_name="${finger3_name}"
+        collision="${collision}"
+        mesh_offset_rpy="${link_finger3_mesh_offset}"
+        parent="${prefix}${hand_name}"
+        prefix="${prefix}"
+        joint_type="${joint_finger3_base_type}"
+        joint_origin_xyz="${joint_finger3_base_origin_xyz}"
+        joint_origin_rpy="${joint_finger3_base_origin_rpy}"
+        joint_axis_xyz="${joint_finger3_base_axis_xyz}"
+        gazebo_preserve_fixed_joint="${gazebo_preserve_fixed_joint}"
+        />
+        <!-- FINGER 4 -->
+        <xacro:unless value="${nbFingers == 3}">
+            <xacro:fingrip_finger
+            finger_name="${finger4_name}"
+            collision="${collision}"
+            mesh_offset_rpy="${link_finger4_mesh_offset}"
+            parent="${prefix}${hand_name}"
+            prefix="${prefix}"
+            joint_type="${joint_finger4_base_type}"
+            joint_origin_xyz="${joint_finger4_base_origin_xyz}"
+            joint_origin_rpy="${joint_finger4_base_origin_rpy}"
+            joint_axis_xyz="${joint_finger4_base_axis_xyz}"
+            gazebo_preserve_fixed_joint="${gazebo_preserve_fixed_joint}"
+            />
+        </xacro:unless>
     <!-- End effector -->
     <xacro:fingrip_virtual_link
