Commit message: ADD: change panda arm to Kuka (OK), (WIP) change the gripper

File: fingrip_description/urdf/fingrip_inertial.xacro (robot description, xacro)
@@ -5,14 +5,34 @@
   <!-- Properties -->
   <!--            -->
-  <xacro:property name="link0_mesh" value="link0"/>
-  <xacro:property name="link1_mesh" value="link1"/>
-  <xacro:property name="link2_mesh" value="link2"/>
-  <xacro:property name="link3_mesh" value="link3"/>
-  <xacro:property name="link4_mesh" value="link4"/>
-  <xacro:property name="link5_mesh" value="link5"/>
-  <xacro:property name="link6_mesh" value="link6"/>
-  <xacro:property name="link7_mesh" value="link7"/>
-  <xacro:property name="hand_mesh" value="hand"/>
-  <xacro:property name="finger_mesh" value="finger"/>
+  <!--    Arm     -->
+  <xacro:property name="link0_mesh" value="arm/link0"/>
+  <xacro:property name="link1_mesh" value="arm/link1"/>
+  <xacro:property name="link2_mesh" value="arm/link2"/>
+  <xacro:property name="link3_mesh" value="arm/link3"/>
+  <xacro:property name="link4_mesh" value="arm/link4"/>
+  <xacro:property name="link5_mesh" value="arm/link5"/>
+  <xacro:property name="link6_mesh" value="arm/link6"/>
+  <xacro:property name="link7_mesh" value="arm/link7"/>
+  <!--  Fingers   -->
+  <xacro:property name="palm_base_mesh_path" value="gripper/paume/base_hand_paume"/>
+  <xacro:property name="case_mesh_path" value="gripper/case/case_"/>
+  <xacro:property name="base_mesh" value="gripper/base_finger/base_finger"/>
+  <xacro:property name="proximal_mesh_path" value="gripper/proximal/"/>
+  <xacro:property name="intermediaire_mesh_path" value="gripper/intermediaire/"/>
+  <xacro:property name="distal_mesh_path" value="gripper/distal/"/>
+  <xacro:property name="long_prefix" value="long/"/>
+  <xacro:property name="short_prefix" value="short/"/>
+  <xacro:property name="proximal_mesh_name" value="proximal"/>
+  <xacro:property name="intermediaire_mesh_name" value="intermediaire"/>
+  <xacro:property name="distal_mesh_name" value="distal"/>
+  <!-- Model changes -->
+  <!-- 3 fingers -->
+  <xacro:property name="f3_suffix" value="3D"/>
+  <!-- 4 fingers -->
+  <xacro:property name="f4_suffix" value="4D"/>
+  <!-- Model 1 -->
+  <xacro:property name="model1_suffix" value="1"/>
+  <!-- Model 2 -->
+  <xacro:property name="model2_suffix" value="2"/>
   <!--       -->
   <!-- Macro -->
@@ -25,5 +45,5 @@
     <xacro:if value="${mesh == link0_mesh}">
       <inertial>
-        <origin xyz="-0.025566 -2.87883e-05 0.057332" rpy="${mesh_offset_rpy}"/>
+        <origin xyz="-0.1 0 0.07" rpy="${mesh_offset_rpy}"/>
         <mass value="2.814271300104062"/>
         <inertia ixx="0.0075390636364814695" iyy="0.010508017427382959" izz="0.009864933638708275" ixy="-1.5053124574783335e-05" ixz="-0.0012144328835738973" iyz="1.0434803501032979e-05"/>
@@ -32,5 +52,5 @@
     <xacro:if value="${mesh == link1_mesh}">
       <inertial>
-        <origin xyz="-3.72212e-09 -0.0324958 -0.0675818" rpy="${mesh_offset_rpy}"/>
+        <origin xyz="0 -0.03 0.12" rpy="${mesh_offset_rpy}"/>
         <mass value="2.6433170427227215"/>
         <inertia ixx="0.017405076982879724" iyy="0.015352077935781732" izz="0.005987891663073857" ixy="-8.687986369621078e-09" ixz="-1.6277819062920423e-08" iyz="0.004510855959102245"/>
@@ -39,5 +59,5 @@
     <xacro:if value="${mesh == link2_mesh}">
       <inertial>
-        <origin xyz="3.17833e-07 -0.06861 0.0322285" rpy="${mesh_offset_rpy}"/>
+        <origin xyz="0.00029 0.059   0.042" rpy="${mesh_offset_rpy}"/>
         <mass value="2.6652755331661186"/>
         <inertia ixx="0.01778694005635383" iyy="0.006044133867952844" izz="0.01571095500455695" ixy="8.70635625879119e-08" ixz="3.752072058394008e-08" iyz="-0.004599490295490376"/>
@@ -46,5 +66,5 @@
     <xacro:if value="${mesh == link3_mesh}">
       <inertial>
-        <origin xyz="0.0469893 0.0316374 -0.031704" rpy="${mesh_offset_rpy}"/>
+        <origin xyz="0   0.03 0.13" rpy="${mesh_offset_rpy}"/>
         <mass value="2.3293714829045733"/>
         <inertia ixx="0.0075496764161139766" iyy="0.009680676080191398" izz="0.007944557422008086" ixy="-0.0024320464513492225" ixz="-0.003250815048103007" iyz="-0.0021316282421730694"/>
@@ -53,5 +73,5 @@
     <xacro:if value="${mesh == link4_mesh}">
       <inertial>
-        <origin xyz="-0.0360505 0.0337069 0.0319019" rpy="${mesh_offset_rpy}"/>
+        <origin xyz="0 0.067 0.034" rpy="${mesh_offset_rpy}"/>
         <mass value="2.3104763646281508"/>
         <inertia ixx="0.007764568814864828" iyy="0.008015776929980149" izz="0.009955882308071066" ixy="0.003371475204045935" ixz="-0.002343621113168248" iyz="0.0022917526161470624"/>
@@ -60,5 +80,5 @@
     <xacro:if value="${mesh == link5_mesh}">
       <inertial>
-        <origin xyz="-6.12525e-06 0.0610427 -0.104176" rpy="${mesh_offset_rpy}"/>
+        <origin xyz="0.0001 0.021  0.076" rpy="${mesh_offset_rpy}"/>
         <mass value="2.6226426154892004"/>
         <inertia ixx="0.029070538014399377" iyy="0.027638529986528795" izz="0.004251111234400737" ixy="6.208738268725568e-07" ixz="-1.0059151925023392e-05" iyz="-0.007424306477850814"/>
@@ -67,5 +87,5 @@
     <xacro:if value="${mesh == link6_mesh}">
       <inertial>
-        <origin xyz="0.051051 0.00910797 0.0106343" rpy="${mesh_offset_rpy}"/>
+        <origin xyz="0.0 0.00059 0.0004" rpy="${mesh_offset_rpy}"/>
         <mass value="1.5025804886626795"/>
         <inertia ixx="0.002940555801469018" iyy="0.00392105201248677" izz="0.0054115603870960195" ixy="-0.00042391108351381507" ixz="0.000610007735338717" iyz="0.00012647545430836214"/>
@@ -74,10 +94,12 @@
     <xacro:if value="${mesh == link7_mesh}">
       <inertial>
-        <origin xyz="0.0109695 0.0107965 0.0650412" rpy="${mesh_offset_rpy}"/>
+        <origin xyz="0.0 0.0 0.02" rpy="${mesh_offset_rpy}"/>
         <mass value="0.5237668134788256"/>
         <inertia ixx="0.0008621467959726535" iyy="0.0008613100184801048" izz="0.0006961139396618219" ixy="-0.00011871071570425467" ixz="3.866602604509339e-05" iyz="-9.057841649422724e-05"/>
       </inertial>
     </xacro:if>
-    <xacro:if value="${mesh == hand_mesh}">
+    <!-- TO DO -->
+    <!-- PALM BASE -->
+    <xacro:if value="${mesh == palm_base_mesh_path+'1'}">
       <inertial>
         <origin xyz="-6.7624e-06 0.00152435 0.0275912" rpy="${mesh_offset_rpy}"/>
@@ -86,5 +108,52 @@
       </inertial>
     </xacro:if>
-    <xacro:if value="${mesh == finger_mesh}">
+    <xacro:if value="${mesh == palm_base_mesh_path+'2'}">
+      <inertial>
+        <origin xyz="-6.7624e-06 0.00152435 0.0275912" rpy="${mesh_offset_rpy}"/>
+        <mass value="0.14060765127978503"/>
+        <inertia ixx="0.0005365450414352072" iyy="7.70511954783727e-05" izz="0.0004938176882694914" ixy="1.7911952957732454e-08" ixz="-2.320071910601251e-08" iyz="4.681149945315967e-08"/>
+      </inertial>
+    </xacro:if>
+    <!-- PALM CASE -->
+    <xacro:if value="${mesh == case_mesh_path+'3D'}">
+      <inertial>
+        <origin xyz="-6.7624e-06 0.00152435 0.0275912" rpy="${mesh_offset_rpy}"/>
+        <mass value="0.14060765127978503"/>
+        <inertia ixx="0.0005365450414352072" iyy="7.70511954783727e-05" izz="0.0004938176882694914" ixy="1.7911952957732454e-08" ixz="-2.320071910601251e-08" iyz="4.681149945315967e-08"/>
+      </inertial>
+    </xacro:if>
+    <xacro:if value="${mesh == case_mesh_path+'4D'}">
+      <inertial>
+        <origin xyz="-6.7624e-06 0.00152435 0.0275912" rpy="${mesh_offset_rpy}"/>
+        <mass value="0.14060765127978503"/>
+        <inertia ixx="0.0005365450414352072" iyy="7.70511954783727e-05" izz="0.0004938176882694914" ixy="1.7911952957732454e-08" ixz="-2.320071910601251e-08" iyz="4.681149945315967e-08"/>
+      </inertial>
+    </xacro:if>
+    <!-- BASE FINGER -->
+    <xacro:if value="${mesh == base_mesh}">
+      <inertial>
+        <origin xyz="-6.2561e-06 0.00227781 -0.0277116" rpy="${mesh_offset_rpy}"/>
+        <mass value="0.2238453537819424"/>
+        <inertia ixx="6.74804167363695e-05" iyy="6.627189221641395e-05" izz="1.550396267804825e-05" ixy="-4.1027443646025676e-09" ixz="1.8693673970152995e-08" iyz="1.1967548474390802e-05"/>
+      </inertial>
+    </xacro:if>
+    <!-- PROXIMAL FINGER -->
+    <xacro:if value="${mesh == proximal_mesh_path+short_prefix+proximal_mesh_name}">
+      <inertial>
+        <origin xyz="-6.2561e-06 0.00227781 -0.0277116" rpy="${mesh_offset_rpy}"/>
+        <mass value="0.2238453537819424"/>
+        <inertia ixx="6.74804167363695e-05" iyy="6.627189221641395e-05" izz="1.550396267804825e-05" ixy="-4.1027443646025676e-09" ixz="1.8693673970152995e-08" iyz="1.1967548474390802e-05"/>
+      </inertial>
+    </xacro:if>
+    <!-- INTERMEDIAIRE FINGER -->
+    <xacro:if value="${mesh == intermediaire_mesh_path+short_prefix+intermediaire_mesh_name}">
+      <inertial>
+        <origin xyz="-6.2561e-06 0.00227781 -0.0277116" rpy="${mesh_offset_rpy}"/>
+        <mass value="0.2238453537819424"/>
+        <inertia ixx="6.74804167363695e-05" iyy="6.627189221641395e-05" izz="1.550396267804825e-05" ixy="-4.1027443646025676e-09" ixz="1.8693673970152995e-08" iyz="1.1967548474390802e-05"/>
+      </inertial>
+    </xacro:if>
+    <!-- DISTAL FINGER -->
+    <xacro:if value="${mesh == distal_mesh_path+short_prefix+distal_mesh_name}">
       <inertial>
         <origin xyz="-6.2561e-06 0.00227781 -0.0277116" rpy="${mesh_offset_rpy}"/>

File: fingrip_description/urdf/fingrip_utils.xacro (robot description, xacro)
@@ -17,4 +17,5 @@
     mesh_offset_rpy:=${mesh_offset_rpy}
     gazebo_self_collide:=false
+    color:=Grey
   ">
     <link name="${link_name}">
@@ -22,6 +23,7 @@
         <origin xyz="0 0 0" rpy="${mesh_offset_rpy}"/>
         <geometry>
-          <mesh filename="package://fingrip_description/meshes/visual/${mesh}.dae"/>
+          <mesh filename="package://fingrip_description/meshes/visual/${mesh}.stl"/>
         </geometry>
+        <material name="${color}"/>
       </visual>
       <xacro:if value="${collision}">
