Commit message: MOD: passage de panda à fingrip, modifications des urdf et srdf (sans prise en compte des paramètres dynamiques et de certaines limitations)

File: fingrip_description/urdf/fingrip.urdf.xacro (robot description, xacro)
@@ -41,9 +41,9 @@
   <!-- Flag to preserve fixed joints and prevent lumping when generating SDF for Gazebo -->
   <xacro:arg name="gazebo_preserve_fixed_joint" default="false"/>
+  <!-- Flag to use underactuation model -->
+  <xacro:arg name="underactuation" default="true"/>
+  <!-- Flag to use long or short fingers model  -->
+  <xacro:arg name="longFingertip" default="false"/>
   <!-- Flag to use 3 or 4 fingers model  -->
-  <xacro:arg name="underactuation" default="true"/>
-  <!-- Flag to use underactuation model -->
-  <xacro:arg name="longFingertip" default="false"/>
-  <!-- Flag to use long or short fingers model  -->
   <xacro:arg name="nbFingers" default="3"/>
   <!-- Flag to use small or bigger palm size  -->
@@ -60,5 +60,5 @@
   <xacro:property name="origin_rpy" value="0 0 0"/>
   <!-- Offset of gripper with respect to wrist flange -->
-  <xacro:property name="gripper_offset_xyz" value="0 0 0"/>
+  <xacro:property name="gripper_offset_xyz" value="0 0 0.0"/>
   <xacro:property name="gripper_offset_rpy" value="0 0 0"/>
   <!-- Import Rviz colors -->

File: fingrip_description/urdf/fingrip_arm.xacro (robot description, xacro)
@@ -114,6 +114,6 @@
   <xacro:property name="link7_color" value="Grey"/>
   <xacro:property name="wrist_flange_name" value="link8"/>
-  <xacro:property name="wrist_flange_origin_xyz" value="0 0 0.107"/>
-  <xacro:property name="wrist_flange_origin_rpy" value="0 0 ${-pi/4}"/>
+  <xacro:property name="wrist_flange_origin_xyz" value="0 0 0.132936"/>
+  <xacro:property name="wrist_flange_origin_rpy" value="0 0 0"/>
   <!--       -->
   <!-- Macro -->

File: fingrip_description/urdf/fingrip_finger.xacro (robot description, xacro)
@@ -20,23 +20,24 @@
   <xacro:property name="joint_friction" value="0.4"/>
   <xacro:property name="link_mu" value="1.13"/>
+  <xacro:property name="joint_other_type" value="revolute"/>
   <!-- Joint dependent properties -->
   <!-- Base -->
   <xacro:property name="joint_base_lower_limit" value="0"/>
-  <xacro:property name="joint_base_upper_limit" value="0.04"/>
+  <xacro:property name="joint_base_upper_limit" value="${pi/2}"/>
   <!-- Proximal -->
-  <xacro:property name="joint_proximal_lower_limit" value="0"/>
-  <xacro:property name="joint_proximal_upper_limit" value="0.04"/>
+  <xacro:property name="joint_proximal_lower_limit" value="-1.3"/>
+  <xacro:property name="joint_proximal_upper_limit" value="0.31416"/>
   <xacro:property name="joint_proximal_origin_xyz" value="0 0 0.0584"/>
   <xacro:property name="joint_proximal_origin_rpy" value="0 0 0"/>
   <xacro:property name="joint_proximal_axis_xyz" value="0 1 0"/>
   <!-- Intermediaire -->
-  <xacro:property name="joint_intermediaire_lower_limit" value="0"/>
-  <xacro:property name="joint_intermediaire_upper_limit" value="0.04"/>
+  <xacro:property name="joint_intermediaire_lower_limit" value="-0.5"/>
+  <xacro:property name="joint_intermediaire_upper_limit" value="1.0472"/>
   <xacro:property name="joint_intermediaire_origin_xyz" value="0 0 0.0584"/>
   <xacro:property name="joint_intermediaire_origin_rpy" value="0 0 0"/>
   <xacro:property name="joint_intermediaire_axis_xyz" value="0 1 0"/>
   <!-- Distal -->
-  <xacro:property name="joint_distal_lower_limit" value="0"/>
-  <xacro:property name="joint_distal_upper_limit" value="0.04"/>
+  <xacro:property name="joint_distal_lower_limit" value="-0.5"/>
+  <xacro:property name="joint_distal_upper_limit" value="1.0472"/>
   <xacro:property name="joint_distal_origin_xyz" value="0 0 0.0584"/>
   <xacro:property name="joint_distal_origin_rpy" value="0 0 0"/>
@@ -57,4 +58,6 @@
     joint_origin_rpy
     joint_axis_xyz:=unset
+    joint_lower_limit:=${joint_base_lower_limit}
+    joint_upper_limit:=${joint_base_upper_limit}
     gazebo_preserve_fixed_joint:=false
   ">
@@ -69,6 +72,6 @@
         joint_origin_rpy="${joint_origin_rpy}"
         joint_axis_xyz="${joint_axis_xyz}"
-        joint_lower_limit="${joint_base_lower_limit}"
-        joint_upper_limit="${joint_base_upper_limit}"
+        joint_lower_limit="${joint_lower_limit}"
+        joint_upper_limit="${joint_upper_limit}"
         joint_velocity_limit="${joint_velocity_limit}"
         joint_torque_limit="${joint_torque_limit}"
@@ -85,4 +88,5 @@
         />
         <!-- PROXIMAL limb -->
+        <!--
         <xacro:fingrip_joint
         parent="${prefix}${finger_name}${base_prefix}${link_prefix}"
@@ -108,5 +112,7 @@
         mesh_offset_rpy="${mesh_offset_rpy}"
         />
+        -->
         <!-- INTERMEDIAIRE limb -->
+        <!--
         <xacro:fingrip_joint
         parent="${prefix}${finger_name}${proximal_prefix}${link_prefix}"
@@ -131,5 +137,7 @@
         mu="${link_mu}"
         />
+        -->
         <!-- DISTAL limb -->
+        <!--
         <xacro:fingrip_joint
         parent="${prefix}${finger_name}${intermediaire_prefix}${link_prefix}"
@@ -154,4 +162,5 @@
         mu="${link_mu}"
         />
+        -->
     </xacro:macro>
 </robot>

File: fingrip_description/urdf/fingrip_gripper.xacro (robot description, xacro)
@@ -11,30 +11,36 @@
   <!-- Properties -->
   <!--            -->
-  <!-- WRIST -->
+  <!-- ROS CONTROL -->
+  <xacro:property name="ros2control_name" value="fingrip_gripper_system"/>
+  <!--    WRIST   -->
   <xacro:property name="joint_wrist_name" value="joint_wrist"/>
   <xacro:property name="joint_wrist_type" value="fixed"/>
   <xacro:property name="hand_name" value="hand"/>
   <xacro:property name="hand_mu" value="0.85"/>
+  <!-- End-Effector -->
+  <xacro:property name="ee_name" value="hand_tcp"/>
+  <xacro:property name="ee_origin_xyz" value="0 0 0.12"/>
+  <xacro:property name="ee_origin_rpy" value="0 0 0"/>
   <!-- Finger dependent properties -->
   <!-- FINGER 1 -->
   <xacro:property name="finger1_name" value="finger1"/>
   <xacro:property name="joint_finger1_base_type" value="revolute"/>
-  <xacro:property name="joint_finger1_base_origin_xyz" value="0 0 0.0584"/>
-  <xacro:property name="joint_finger1_base_origin_rpy" value="0 0 0"/>
-  <xacro:property name="joint_finger1_base_axis_xyz" value="0 1 0"/>
+  <xacro:property name="joint_finger1_base_origin_xyz" value="0.054 0.054 0.09885097"/>
+  <xacro:property name="joint_finger1_base_origin_rpy" value="0 ${-pi/2} ${-pi}"/>
+  <xacro:property name="joint_finger1_base_axis_xyz" value="1 0 0"/>
   <xacro:property name="link_finger1_mesh_offset" value="0 0 0"/>
   <!-- FINGER 2 -->
   <xacro:property name="finger2_name" value="finger2"/>
   <xacro:property name="joint_finger2_base_type" value="revolute"/>
-  <xacro:property name="joint_finger2_base_origin_xyz" value="0 0 0.0584"/>
-  <xacro:property name="joint_finger2_base_origin_rpy" value="0 0 0"/>
-  <xacro:property name="joint_finger2_base_axis_xyz" value="0 1 0"/>
+  <xacro:property name="joint_finger2_base_origin_xyz" value="0.054 -0.054 0.09885097"/>
+  <xacro:property name="joint_finger2_base_origin_rpy" value="${pi} ${-pi/2} ${pi}"/>
+  <xacro:property name="joint_finger2_base_axis_xyz" value="1 0 0"/>
   <xacro:property name="link_finger2_mesh_offset" value="0 0 0"/>
   <!-- FINGER 3 -->
   <xacro:property name="finger3_name" value="finger3"/>
   <xacro:property name="joint_finger3_base_type" value="fixed"/>
-  <xacro:property name="joint_finger3_base_origin_xyz" value="0 0 0.0584"/>
-  <xacro:property name="joint_finger3_base_origin_rpy" value="0 0 0"/>
-  <xacro:property name="joint_finger3_base_axis_xyz" value="0 1 0"/>
+  <xacro:property name="joint_finger3_base_origin_xyz" value="-0.04398 0 0.09885097"/>
+  <xacro:property name="joint_finger3_base_origin_rpy" value="${-pi/2} ${-pi/2} 0"/>
+  <xacro:property name="joint_finger3_base_axis_xyz" value="0 0 0"/>
   <xacro:property name="link_finger3_mesh_offset" value="0 0 0"/>
   <!-- FINGER 4 -->
@@ -43,5 +49,5 @@
   <xacro:property name="joint_finger4_base_origin_xyz" value="0 0 0.0584"/>
   <xacro:property name="joint_finger4_base_origin_rpy" value="0 0 0"/>
-  <xacro:property name="joint_finger4_base_axis_xyz" value="0 1 0"/>
+  <xacro:property name="joint_finger4_base_axis_xyz" value="0 0 0"/>
   <xacro:property name="link_finger4_mesh_offset" value="0 0 0"/>
   <!--       -->
@@ -91,4 +97,6 @@
         joint_origin_rpy="${joint_finger1_base_origin_rpy}"
         joint_axis_xyz="${joint_finger1_base_axis_xyz}"
+        joint_lower_limit="${-joint_base_upper_limit}"
+        joint_upper_limit="${-joint_base_lower_limit}"
         gazebo_preserve_fixed_joint="${gazebo_preserve_fixed_joint}"
         />
@@ -144,5 +152,30 @@
     <!-- ROS 2 control -->
     <xacro:if value="${ros2_control}">
-      <xacro:ros2_control_fingrip_gripper prefix="${prefix}" plugin="${ros2_control_plugin}" command_interface="${ros2_control_command_interface}"/>
+      <ros2_control name="${ros2control_name}" type="system">
+        <xacro:ros2_control_fingrip_gripper
+        prefix="${prefix}"
+        plugin="${ros2_control_plugin}"
+        command_interface="${ros2_control_command_interface}"
+        finger_name="${finger1_name}"/>
+        <xacro:ros2_control_fingrip_gripper
+        prefix="${prefix}"
+        plugin="${ros2_control_plugin}"
+        command_interface="${ros2_control_command_interface}"
+        finger_name="${finger2_name}"/>
+        <!--
+        <xacro:ros2_control_fingrip_gripper
+        prefix="${prefix}"
+        plugin="${ros2_control_plugin}"
+        command_interface="${ros2_control_command_interface}"
+        finger_name="${finger3_name}"/>
+        -->
+        <xacro:unless value="${nbFingers == 3}">
+          <xacro:ros2_control_fingrip_gripper
+          prefix="${prefix}"
+          plugin="${ros2_control_plugin}"
+          command_interface="${ros2_control_command_interface}"
+          finger_name="${finger4_name}"/>
+        </xacro:unless>
+      </ros2_control>
     </xacro:if>
   </xacro:macro>

File: fingrip_description/urdf/fingrip_inertial.xacro (robot description, xacro)
@@ -28,7 +28,7 @@
   <!-- Model changes -->
   <!-- 3 fingers -->
-  <xacro:property name="f3_suffix" value="3D"/>
+  <xacro:property name="f3_suffix" value="3d"/>
   <!-- 4 fingers -->
-  <xacro:property name="f4_suffix" value="4D"/>
+  <xacro:property name="f4_suffix" value="4d"/>
   <!-- Model 1 -->
   <xacro:property name="model1_suffix" value="1"/>
@@ -103,5 +103,5 @@
     <xacro:if value="${mesh == palm_base_mesh_path+'1'}">
       <inertial>
-        <origin xyz="-6.7624e-06 0.00152435 0.0275912" rpy="${mesh_offset_rpy}"/>
+        <origin xyz="0.00 0.0 -0.04835" rpy="${mesh_offset_rpy}"/>
         <mass value="0.14060765127978503"/>
         <inertia ixx="0.0005365450414352072" iyy="7.70511954783727e-05" izz="0.0004938176882694914" ixy="1.7911952957732454e-08" ixz="-2.320071910601251e-08" iyz="4.681149945315967e-08"/>
@@ -116,5 +116,5 @@
     </xacro:if>
     <!-- PALM CASE -->
-    <xacro:if value="${mesh == case_mesh_path+'3D'}">
+    <xacro:if value="${mesh == case_mesh_path+'3d'}">
       <inertial>
         <origin xyz="-6.7624e-06 0.00152435 0.0275912" rpy="${mesh_offset_rpy}"/>
@@ -123,5 +123,5 @@
       </inertial>
     </xacro:if>
-    <xacro:if value="${mesh == case_mesh_path+'4D'}">
+    <xacro:if value="${mesh == case_mesh_path+'4d'}">
       <inertial>
         <origin xyz="-6.7624e-06 0.00152435 0.0275912" rpy="${mesh_offset_rpy}"/>

File: fingrip_description/urdf/fingrip_palm.xacro (robot description, xacro)
@@ -12,5 +12,5 @@
   <xacro:property name="joint_palm_name" value="joint_palm"/>
   <xacro:property name="joint_palm_type" value="fixed"/>
-  <xacro:property name="palm_origin_xyz" value="0 0 0"/>
+  <xacro:property name="palm_origin_xyz" value="0 0 0.013"/>
   <xacro:property name="palm_origin_rpy" value="0 0 0"/>
   <!--       -->
@@ -46,5 +46,5 @@
         <xacro:fingrip_link
         link_name="${prefix}${hand_name}"
-        mesh="${palm_base_mesh_path}1"
+        mesh="${palm_base_mesh_path}${model1_suffix}"
         collision="${collision}"
         mu="${mu}"
@@ -63,5 +63,5 @@
         <xacro:fingrip_link
         link_name="${prefix}${hand_name}"
-        mesh="${palm_base_mesh_path}2"
+        mesh="${palm_base_mesh_path}${model2_suffix}"
         collision="${collision}"
         mu="${mu}"
@@ -81,5 +81,5 @@
         <xacro:fingrip_link
         link_name="${prefix}${palm_name}"
-        mesh="${case_mesh_path}3D"
+        mesh="${case_mesh_path}${f3_suffix}"
         collision="${collision}"
         mu="${mu}"
@@ -98,5 +98,5 @@
         <xacro:fingrip_link
         link_name="${prefix}${palm_name}"
-        mesh="${case_mesh_path}4D"
+        mesh="${case_mesh_path}${f4_suffix}"
         collision="${collision}"
         mu="${mu}"

File: fingrip_description/urdf/fingrip_utils.xacro (robot description, xacro)
@@ -122,5 +122,5 @@
       </transmission>
     </xacro:unless>
-    <!-- Spring stiffness and reference for non-fifex joint -->
+    <!-- Spring stiffness and reference for non-fifed joint -->
     <xacro:unless value="${joint_type == 'fixed'}">
       <gazebo reference="${joint_name}">

File: fingrip_moveit_config/srdf/fingrip.srdf.xacro (robot description, xacro)
@@ -34,11 +34,19 @@
   <disable_collisions link1="${prefix_gripper}hand" link2="${prefix_arm}link6" reason="Never"/>
   <disable_collisions link1="${prefix_gripper}hand" link2="${prefix_arm}link7" reason="Adjacent"/>
-  <disable_collisions link1="${prefix_gripper}leftfinger" link2="${prefix_arm}link3" reason="Never"/>
-  <disable_collisions link1="${prefix_gripper}leftfinger" link2="${prefix_arm}link4" reason="Never"/>
-  <disable_collisions link1="${prefix_gripper}leftfinger" link2="${prefix_arm}link6" reason="Never"/>
-  <disable_collisions link1="${prefix_gripper}leftfinger" link2="${prefix_arm}link7" reason="Never"/>
-  <disable_collisions link1="${prefix_arm}link3" link2="${prefix_gripper}rightfinger" reason="Never"/>
-  <disable_collisions link1="${prefix_arm}link4" link2="${prefix_gripper}rightfinger" reason="Never"/>
-  <disable_collisions link1="${prefix_arm}link6" link2="${prefix_gripper}rightfinger" reason="Never"/>
-  <disable_collisions link1="${prefix_arm}link7" link2="${prefix_gripper}rightfinger" reason="Never"/>
+  <disable_collisions link1="${prefix_gripper}palm" link2="${prefix_arm}link3" reason="Never"/>
+  <disable_collisions link1="${prefix_gripper}palm" link2="${prefix_arm}link4" reason="Never"/>
+  <disable_collisions link1="${prefix_gripper}palm" link2="${prefix_arm}link6" reason="Never"/>
+  <disable_collisions link1="${prefix_gripper}palm" link2="${prefix_arm}link7" reason="Never"/>
+  <disable_collisions link1="${prefix_gripper}finger1_base_link" link2="${prefix_arm}link3" reason="Never"/>
+  <disable_collisions link1="${prefix_gripper}finger1_base_link" link2="${prefix_arm}link4" reason="Never"/>
+  <disable_collisions link1="${prefix_gripper}finger1_base_link" link2="${prefix_arm}link6" reason="Never"/>
+  <disable_collisions link1="${prefix_gripper}finger1_base_link" link2="${prefix_arm}link7" reason="Never"/>
+  <disable_collisions link1="${prefix_gripper}finger2_base_link" link2="${prefix_arm}link3" reason="Never"/>
+  <disable_collisions link1="${prefix_gripper}finger2_base_link" link2="${prefix_arm}link4" reason="Never"/>
+  <disable_collisions link1="${prefix_gripper}finger2_base_link" link2="${prefix_arm}link6" reason="Never"/>
+  <disable_collisions link1="${prefix_gripper}finger2_base_link" link2="${prefix_arm}link7" reason="Never"/>
+  <disable_collisions link1="${prefix_gripper}finger3_base_link" link2="${prefix_arm}link3" reason="Never"/>
+  <disable_collisions link1="${prefix_gripper}finger3_base_link" link2="${prefix_arm}link4" reason="Never"/>
+  <disable_collisions link1="${prefix_gripper}finger3_base_link" link2="${prefix_arm}link6" reason="Never"/>
+  <disable_collisions link1="${prefix_gripper}finger3_base_link" link2="${prefix_arm}link7" reason="Never"/>
 </robot>

File: fingrip_moveit_config/srdf/fingrip_arm.xacro (robot description, xacro)
@@ -11,4 +11,5 @@
       <chain base_link="${prefix}link0" tip_link="${prefix}hand_tcp"/>
     </group>
+    <!-- Can configurate pos -->
     <group_state group="arm" name="ready">
       <joint name="${prefix}joint1" value="0"/>
@@ -26,6 +27,6 @@
       <joint name="${prefix}joint4" value="0"/>
       <joint name="${prefix}joint5" value="0"/>
-      <joint name="${prefix}joint6" value="${pi/2}"/>
-      <joint name="${prefix}joint7" value="${pi/4}"/>
+      <joint name="${prefix}joint6" value="0"/>
+      <joint name="${prefix}joint7" value="0"/>
     </group_state>
     <group_state group="arm" name="transport">

File: fingrip_moveit_config/srdf/fingrip_gripper.xacro (robot description, xacro)
@@ -10,20 +10,27 @@
     <group name="gripper">
       <link name="${prefix}hand"/>
-      <link name="${prefix}leftfinger"/>
-      <link name="${prefix}rightfinger"/>
-      <joint name="${prefix}finger_joint1"/>
-      <joint name="${prefix}finger_joint2"/>
+      <link name="${prefix}palm"/>
+      <link name="${prefix}finger1_base_link"/>
+      <link name="${prefix}finger2_base_link"/>
+      <link name="${prefix}finger3_base_link"/>
+      <joint name="${prefix}finger1_base_joint"/>
+      <joint name="${prefix}finger2_base_joint"/>
     </group>
     <group_state name="open" group="gripper">
-      <joint name="${prefix}finger_joint1" value="0.04"/>
-      <joint name="${prefix}finger_joint2" value="0.04"/>
+      <joint name="${prefix}finger1_base_joint" value="-${pi/2}"/>
+      <joint name="${prefix}finger2_base_joint" value="${pi/2}"/>
     </group_state>
     <group_state name="close" group="gripper">
-      <joint name="${prefix}finger_joint1" value="0.0"/>
-      <joint name="${prefix}finger_joint2" value="0.0"/>
+      <joint name="${prefix}finger1_base_joint" value="0.0"/>
+      <joint name="${prefix}finger2_base_joint" value="0.0"/>
     </group_state>
-    <disable_collisions link1="${prefix}hand" link2="${prefix}leftfinger" reason="Adjacent"/>
-    <disable_collisions link1="${prefix}hand" link2="${prefix}rightfinger" reason="Adjacent"/>
-    <disable_collisions link1="${prefix}leftfinger" link2="${prefix}rightfinger" reason="Default"/>
+    <disable_collisions link1="${prefix}hand" link2="${prefix}palm" reason="Adjacent"/>
+    <disable_collisions link1="${prefix}hand" link2="${prefix}finger1_base_link" reason="Adjacent"/>
+    <disable_collisions link1="${prefix}palm" link2="${prefix}finger1_base_link" reason="Adjacent"/>
+    <disable_collisions link1="${prefix}hand" link2="${prefix}finger2_base_link" reason="Adjacent"/>
+    <disable_collisions link1="${prefix}palm" link2="${prefix}finger2_base_link" reason="Adjacent"/>
+    <disable_collisions link1="${prefix}hand" link2="${prefix}finger3_base_link" reason="Adjacent"/>
+    <disable_collisions link1="${prefix}palm" link2="${prefix}finger3_base_link" reason="Adjacent"/>
+    <!-- <disable_collisions link1="${prefix}leftfinger" link2="${prefix}rightfinger" reason="Default"/> -->
   </xacro:macro>
 </robot>
