Commit message: ADD: new controller in xacro file with abduction underactuated (WIP)

File: fingrip_description/urdf/fingrip.urdf.xacro (robot description, xacro)
@@ -43,4 +43,6 @@
   <!-- Flag to use underactuation model -->
   <xacro:arg name="underactuation" default="true"/>
+  <!-- Flag to use underactuated abduction model -->
+  <xacro:arg name="abduction" default="true"/>
   <!-- Flag to use long or short fingers model  -->
   <xacro:arg name="longFingertip" default="false"/>
@@ -108,5 +110,6 @@
       ros2_control_command_interface="$(arg ros2_control_command_interface)"
       gazebo_preserve_fixed_joint="$(arg gazebo_preserve_fixed_joint)"
-      underactuation="$(arg underactuation)"
+      underactuated_fingers="$(arg underactuation)"
+      abduction="$(arg abduction)"
       longFingertip="$(arg longFingertip)"
       nbFingers="$(arg nbFingers)"

File: fingrip_description/urdf/fingrip_arm.xacro (robot description, xacro)
@@ -135,4 +135,5 @@
     ros2_control_command_interface:=effort
     gazebo_preserve_fixed_joint:=false
+    arm:=true
   ">
     <!-- Base -->
@@ -145,4 +146,5 @@
     joint_origin_rpy="${origin_rpy}"
     gazebo_preserve_fixed_joint="${gazebo_preserve_fixed_joint}"
+    arm="${arm}"
     />
     <xacro:fingrip_link
@@ -173,4 +175,5 @@
     safety_k_velocity="${safety_k_velocity}"
     gazebo_preserve_fixed_joint="${gazebo_preserve_fixed_joint}"
+    arm="${arm}"
     />
     <xacro:fingrip_link
@@ -201,4 +204,5 @@
     safety_k_velocity="${safety_k_velocity}"
     gazebo_preserve_fixed_joint="${gazebo_preserve_fixed_joint}"
+    arm="${arm}"
     />
     <xacro:fingrip_link
@@ -229,4 +233,5 @@
     safety_k_velocity="${safety_k_velocity}"
     gazebo_preserve_fixed_joint="${gazebo_preserve_fixed_joint}"
+    arm="${arm}"
     />
     <xacro:fingrip_link
@@ -257,4 +262,5 @@
     safety_k_velocity="${safety_k_velocity}"
     gazebo_preserve_fixed_joint="${gazebo_preserve_fixed_joint}"
+    arm="${arm}"
     />
     <xacro:fingrip_link
@@ -285,4 +291,5 @@
     safety_k_velocity="${safety_k_velocity}"
     gazebo_preserve_fixed_joint="${gazebo_preserve_fixed_joint}"
+    arm="${arm}"
     />
     <xacro:fingrip_link
@@ -313,4 +320,5 @@
     safety_k_velocity="${safety_k_velocity}"
     gazebo_preserve_fixed_joint="${gazebo_preserve_fixed_joint}"
+    arm="${arm}"
     />
     <xacro:fingrip_link
@@ -341,4 +349,5 @@
     safety_k_velocity="${safety_k_velocity}"
     gazebo_preserve_fixed_joint="${gazebo_preserve_fixed_joint}"
+    arm="${arm}"
     />
     <xacro:fingrip_link

File: fingrip_description/urdf/fingrip_gripper.xacro (robot description, xacro)
@@ -8,4 +8,5 @@
   <xacro:include filename="$(find fingrip_description)/urdf/fingrip_finger.xacro"/>
   <xacro:include filename="$(find fingrip_description)/urdf/fingrip_palm.xacro"/>
+  <xacro:include filename="$(find fingrip_description)/urdf/fingrip_transmission.xacro"/>
   <!--            -->
   <!-- Properties -->
@@ -66,5 +67,6 @@
     ros2_control_command_interface:=effort
     gazebo_preserve_fixed_joint:=false
-    underactuation:=true
+    underactuated_fingers:=true
+    abduction:=true
     longFingertip:=false
     nbFingers:=3
@@ -150,4 +152,21 @@
     gazebo_preserve_fixed_joint="${gazebo_preserve_fixed_joint}"
     />
+    <!-- Transmission gripper -->
+    <!-- Abduction -->
+    <xacro:fingrip_transmission
+      joint1_name="${prefix}${finger1_name}${base_prefix}${joint_prefix}"
+      joint2_name="${prefix}${finger2_name}${base_prefix}${joint_prefix}"
+      underactuation="${abduction}"
+      abduction="true"
+    />
+    <!-- Fingers -->
+    <!--
+    <xacro:fingrip_transmission
+      joint1_name="${prefix}${finger1_name}${base_prefix}${joint_prefix}"
+      joint2_name="${prefix}${finger2_name}${base_prefix}${joint_prefix}"
+      underactuation="${underactuated_fingers}"
+      abduction="false"
+    />
+    -->
     <!-- ROS 2 control -->
     <xacro:if value="${ros2_control}">

File: fingrip_description/urdf/fingrip_utils.xacro (robot description, xacro)
@@ -70,4 +70,5 @@
     gazebo_spring_reference:=0.0
     gazebo_preserve_fixed_joint:=false
+    arm:=false
   ">
     <!-- Make sure limits are set for non-fixed joints -->
@@ -111,16 +112,18 @@
     </joint>
     <!-- Transmission for non-fixed joints -->
-    <xacro:unless value="${joint_type == 'fixed'}">
-      <transmission name="${joint_name}_transmission">
-        <type>transmission_interface/SimpleTransmission</type>
-        <joint name="${joint_name}">
-          <hardwareInterface>hardware_interface/EffortJointInterface</hardwareInterface>
-        </joint>
-        <actuator name="${joint_name}_actuator">
-          <mechanicalReduction>1</mechanicalReduction>
-        </actuator>
-      </transmission>
-    </xacro:unless>
-    <!-- Spring stiffness and reference for non-fifed joint -->
+    <xacro:if value="${arm}">
+      <xacro:unless value="${joint_type == 'fixed'}">
+        <transmission name="${joint_name}_transmission">
+          <type>transmission_interface/SimpleTransmission</type>
+          <joint name="${joint_name}">
+            <hardwareInterface>hardware_interface/EffortJointInterface</hardwareInterface>
+          </joint>
+          <actuator name="${joint_name}_actuator">
+            <mechanicalReduction>1</mechanicalReduction>
+          </actuator>
+        </transmission>
+      </xacro:unless>
+    </xacro:if>
+    <!-- Spring stiffness and reference for non-fixed joint -->
     <xacro:unless value="${joint_type == 'fixed'}">
       <gazebo reference="${joint_name}">
